File: EECD-22-7/untitled.kicad_sch (KiCad schematic)
At the start: 3 parts, among them J1_I2C_Gamma_Sensor? Conn_01x06_Female, U1_Pressure_Sensor? MS5525DSO, U2_Temperature_Sensor? TMP1075D

Commit message: Add files via upload
Parts:
- added U?: MAX485E, symbol Interface_UART:MAX485E
Changed lines of the file:
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@@
 (kicad_sch (version 20211123) (generator eeschema)
   (paper "A4")
+  (symbol (lib_id "Interface_UART:MAX485E") (at 123.19 123.19 0) (unit 1)
+    (in_bom yes) (on_board yes) (fields_autoplaced)
+    (property "Reference" "U?" (id 0) (at 125.2094 107.95 0)
+      (effects (font (size 1.27 1.27)) (justify left))
+    )
+    (property "Value" "MAX485E" (id 1) (at 125.2094 110.49 0)
+      (effects (font (size 1.27 1.27)) (justify left))
+    )
+    (property "Footprint" "" (id 2) (at 123.19 140.97 0)
+      (effects (font (size 1.27 1.27)) hide)
+    )
+    (property "Datasheet" "https://datasheets.maximintegrated.com/en/ds/MAX1487E-MAX491E.pdf" (id 3) (at 123.19 121.92 0)
+      (effects (font (size 1.27 1.27)) hide)
+    )
+    (pin "1")
+    (pin "2")
+    (pin "3")
+    (pin "4")
+    (pin "5")
+    (pin "6")
+    (pin "7")
+    (pin "8")
+  )
   (symbol (lib_id "Sensor_Pressure:MS5525DSO") (at 186.944 83.82 0) (unit 1)
     (in_bom yes) (on_board yes) (fields_autoplaced)
