File: EECD-22-7/_autosave-untitled.kicad_sch (KiCad schematic)
At the start: 5 parts, among them J1_I2C_Gamma_Sensor? Conn_01x06_Female, U1_Pressure_Sensor? MS5525DSO, U2_Temperature_Sensor? TMP1075D, U7 519, U8 MAX485E

Commit message: Add files via upload
Parts:
- removed J1_I2C_Gamma_Sensor?: Conn_01x06_Female, symbol Connector:Conn_01x06_Female
- removed U1_Pressure_Sensor?: MS5525DSO, symbol Sensor_Pressure:MS5525DSO
- removed U2_Temperature_Sensor?: TMP1075D, Package_SO:SO-8_3.9x4.9mm_P1.27mm, symbol Sensor_Temperature:TMP1075D
- removed U7: 519, symbol Analog:519
- removed U8: MAX485E, symbol Interface_UART:MAX485E
- added J1_I2C_Gamma_Sensor?: Conn_01x06_Female, symbol Connector:Conn_01x06_Female
- added U1_Pressure_Sensor?: MS5525DSO, symbol Sensor_Pressure:MS5525DSO
- added U2_Temperature_Sensor?: TMP1075D, Package_SO:SO-8_3.9x4.9mm_P1.27mm, symbol Sensor_Temperature:TMP1075D
- added U?: MAX485E, symbol Interface_UART:MAX485E
Connections:
- new net: U1_Pressure_Sensor?.1 (SIN-), U1_Pressure_Sensor?.3 (SIN-)
- new net: U1_Pressure_Sensor?.11 (SUPPLY+), U1_Pressure_Sensor?.13 (SUPPLY+)
- new net: U1_Pressure_Sensor?.12 (SOUT+), U1_Pressure_Sensor?.14 (SOUT+)
- new net: U1_Pressure_Sensor?.2 (SOUT-), U1_Pressure_Sensor?.4 (SOUT-)
Changed lines of the file:
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@@
 (kicad_sch (version 20211123) (generator eeschema)
   (paper "A4")
-  (symbol (lib_id "Connector:Conn_01x06_Female") (at 140.97 132.08 0) (unit 1)
+  (symbol (lib_id "Interface_UART:MAX485E") (at 86.36 81.28 0) (unit 1)
     (in_bom yes) (on_board yes) (fields_autoplaced)
-    (property "Reference" "J1_I2C_Gamma_Sensor?" (id 0) (at 141.859 132.0799 0)
+    (property "Reference" "U?" (id 0) (at 88.3794 66.04 0)
       (effects (font (size 1.27 1.27)) (justify left))
     )
-    (property "Value" "Conn_01x06_Female" (id 1) (at 141.859 134.6199 0)
+    (property "Value" "MAX485E" (id 1) (at 88.3794 68.58 0)
       (effects (font (size 1.27 1.27)) (justify left))
     )
-    (property "Footprint" "" (id 2) (at 140.97 132.08 0))
-    (property "Datasheet" "~" (id 3) (at 140.97 132.08 0)
+    (property "Footprint" "" (id 2) (at 86.36 99.06 0)
       (effects (font (size 1.27 1.27)) hide)
     )
-    (pin "1")
-    (pin "2")
-    (pin "3")
-    (pin "4")
-    (pin "5")
-    (pin "6")
-  )
-  (symbol (lib_id "Sensor_Temperature:TMP1075D") (at 236.982 125.984 0) (unit 1)
-    (in_bom yes) (on_board yes) (fields_autoplaced)
-    (property "Reference" "U2_Temperature_Sensor?" (id 0) (at 239.0014 115.824 0)
-      (effects (font (size 1.27 1.27)) (justify left))
-    )
-    (property "Value" "TMP1075D" (id 1) (at 239.0014 118.364 0)
-      (effects (font (size 1.27 1.27)) (justify left))
-    )
-    (property "Footprint" "Package_SO:SO-8_3.9x4.9mm_P1.27mm" (id 2) (at 236.982 132.334 0)
-      (effects (font (size 1.27 1.27)) hide)
-    )
-    (property "Datasheet" "https://www.ti.com/lit/gpn/tmp1075" (id 3) (at 236.982 125.984 0)
+    (property "Datasheet" "https://datasheets.maximintegrated.com/en/ds/MAX1487E-MAX491E.pdf" (id 3) (at 86.36 80.01 0)
       (effects (font (size 1.27 1.27)) hide)
     )
@@
     (pin "8")
   )
-  (symbol (lib_id "Interface_UART:MAX485E") (at 140.97 88.9 0) (unit 1)
+  (symbol (lib_id "Sensor_Pressure:MS5525DSO") (at 186.944 83.82 0) (unit 1)
     (in_bom yes) (on_board yes) (fields_autoplaced)
-    (property "Reference" "U8" (id 0) (at 142.9894 73.66 0)
+    (property "Reference" "U1_Pressure_Sensor?" (id 0) (at 188.9634 68.58 0)
       (effects (font (size 1.27 1.27)) (justify left))
     )
-    (property "Value" "MAX485E" (id 1) (at 142.9894 76.2 0)
+    (property "Value" "MS5525DSO" (id 1) (at 188.9634 71.12 0)
       (effects (font (size 1.27 1.27)) (justify left))
     )
-    (property "Footprint" "" (id 2) (at 140.97 106.68 0)
+    (property "Footprint" "" (id 2) (at 186.944 97.79 0)
       (effects (font (size 1.27 1.27)) hide)
     )
-    (property "Datasheet" "https://datasheets.maximintegrated.com/en/ds/MAX1487E-MAX491E.pdf" (id 3) (at 140.97 87.63 0)
-      (effects (font (size 1.27 1.27)) hide)
-    )
-    (pin "1")
-    (pin "2")
-    (pin "3")
-    (pin "4")
-    (pin "5")
-    (pin "6")
-    (pin "7")
-    (pin "8")
-  )
-  (symbol (lib_id "Sensor_Pressure:MS5525DSO") (at 241.554 91.44 0) (unit 1)
-    (in_bom yes) (on_board yes) (fields_autoplaced)
-    (property "Reference" "U1_Pressure_Sensor?" (id 0) (at 243.5734 76.2 0)
-      (effects (font (size 1.27 1.27)) (justify left))
-    )
-    (property "Value" "MS5525DSO" (id 1) (at 243.5734 78.74 0)
-      (effects (font (size 1.27 1.27)) (justify left))
-    )
-    (property "Footprint" "" (id 2) (at 241.554 105.41 0)
-      (effects (font (size 1.27 1.27)) hide)
-    )
-    (property "Datasheet" "https://www.te.com/commerce/DocumentDelivery/DDEController?Action=srchrtrv&DocNm=MS5525DSO&DocType=DS&DocLang=English" (id 3) (at 241.554 107.95 0)
+    (property "Datasheet" "https://www.te.com/commerce/DocumentDelivery/DDEController?Action=srchrtrv&DocNm=MS5525DSO&DocType=DS&DocLang=English" (id 3) (at 186.944 100.33 0)
       (effects (font (size 1.27 1.27)) hide)
     )
@@
     (pin "9")
   )
-  (symbol (lib_id "Analog:519") (at 50.8 91.44 0) (unit 1)
-    (in_bom yes) (on_board no) (fields_autoplaced)
-    (property "Reference" "U7" (id 0) (at 50.8 71.12 0))
-    (property "Value" "519" (id 1) (at 50.8 73.66 0))
-    (property "Footprint" "" (id 2) (at 50.8 91.44 0)
-      (effects (font (size 1.27 1.27) italic) hide)
+  (symbol (lib_id "Sensor_Temperature:TMP1075D") (at 182.372 118.364 0) (unit 1)
+    (in_bom yes) (on_board yes) (fields_autoplaced)
+    (property "Reference" "U2_Temperature_Sensor?" (id 0) (at 184.3914 108.204 0)
+      (effects (font (size 1.27 1.27)) (justify left))
     )
-    (property "Datasheet" "https://apautomatyka.pl/download/dat_519_Huba-Control_en.pdf" (id 3) (at 50.8 72.39 0)
-      (effects (font (size 0.5 0.5)) hide)
+    (property "Value" "TMP1075D" (id 1) (at 184.3914 110.744 0)
+      (effects (font (size 1.27 1.27)) (justify left))
+    )
+    (property "Footprint" "Package_SO:SO-8_3.9x4.9mm_P1.27mm" (id 2) (at 182.372 124.714 0)
+      (effects (font (size 1.27 1.27)) hide)
+    )
+    (property "Datasheet" "https://www.ti.com/lit/gpn/tmp1075" (id 3) (at 182.372 118.364 0)
+      (effects (font (size 1.27 1.27)) hide)
     )
     (pin "1")
+    (pin "2")
     (pin "3")
     (pin "4")
+    (pin "5")
+    (pin "6")
+    (pin "7")
+    (pin "8")
+  )
+  (symbol (lib_id "Connector:Conn_01x06_Female") (at 86.36 124.46 0) (unit 1)
+    (in_bom yes) (on_board yes) (fields_autoplaced)
+    (property "Reference" "J1_I2C_Gamma_Sensor?" (id 0) (at 87.249 124.4599 0)
+      (effects (font (size 1.27 1.27)) (justify left))
+    )
+    (property "Value" "Conn_01x06_Female" (id 1) (at 87.249 126.9999 0)
+      (effects (font (size 1.27 1.27)) (justify left))
+    )
+    (property "Footprint" "" (id 2) (at 86.36 124.46 0))
+    (property "Datasheet" "~" (id 3) (at 86.36 124.46 0)
+      (effects (font (size 1.27 1.27)) hide)
+    )
+    (pin "1")
+    (pin "2")
+    (pin "3")
+    (pin "4")
+    (pin "5")
+    (pin "6")
   )
 )
