File: EECD-22-7/power.kicad_sch (KiCad schematic)
At the start: 2 parts, among them U2 LM25183NGUR, U3 LM5181NGUR

Commit message: Add files via upload
Parts:
- removed U2: LM25183NGUR, symbol Regulator_Controller:LM25183NGUR
- added C10, C4, C6, C7: 10uF, symbol pspice:C
- added C5, C6, C8, C9: 100nF, symbol pspice:C
- added L1: 150uH, symbol Device:L
- added L2: 15uH, symbol Device:L
- added R4: 115kR, symbol Device:R
- added R5, R8: 22kR, symbol Device:R
- added R7: 309kR, symbol Device:R
- added U4: LMR54406DBVR, symbol Regulator_Switching:LM5181NGUR
- U3: value LM5181NGUR -> LMR54406DBVR
Connections:
- net at U3.1 (CB): now also C6.2
- net +BATT: now reaches U3.2 (VIN)
- net +BATT: now also U3.3 (EN), C4.1, C5.1, C7.1, C8.1, U4.2 (VIN), U4.3 (EN)
- net at U3.4 (SW): now also C6.1, L1.1
- net at U3.5 (FB): now also R4.2, R5.1
- net -BATT: now reaches U3.6 (GND)
- net -BATT: now also C10.2, C4.2, C5.2, C6.2, C7.2, C8.2, R5.2, R8.2, U4.6 (GND)
- new net: C9.1, L2.1, U4.4 (SW)
- new net: C9.2, U4.1 (CB)
- new net: R7.2, R8.1, U4.5 (FB)
- new net +12V: C10.1, L2.2, R7.1
- new net +5V: C6.1, L1.2, R4.1

Commit message: Add files via upload
Parts:
- added C11, C14: 10uF, symbol pspice:C
- added C12, C13: 100nF, symbol pspice:C
- added L3: 12uH, symbol Device:L
- added R8: 70kR, symbol Device:R
- added R9: 22kR, symbol Device:R
- added U5: LMR54406DBVR, symbol Regulator_Switching:LM5181NGUR
Connections:
- net +BATT: now also C11.1, C12.1, U5.2 (VIN), U5.3 (EN)
- net -BATT: now also C11.2, C12.2, C14.2, R9.2, U5.6 (GND)
- new net: R8.2, R9.1, U5.5 (FB)
- new net: C13.1, L3.1, U5.4 (SW)
- new net: C13.2, U5.1 (CB)
- new net +3.3V: C14.1, L3.2, R8.1
Other:
- moved on the sheet: C10, C4, C5, C6, C7, C8, C9, L1, L2, R4, R5, R7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

Commit message: Add files via upload
Parts:
- added Q1, Q2: IRF6616, Package_DirectFET:DirectFET_MX, symbol Transistor_FET:IRF6616
- added R20, R?: 10kR, symbol Device:R
Connections:
- net -BATT: now also Q1.1 (D), Q1.3 (S), Q2.1 (D), Q2.3 (S), R20.1, R?.1
- new net peri_power_1: Q1.2 (G), R20.2
- new net peri_power_2: Q2.2 (G), R?.2
Other:
- moved on the sheet: C7, C8

Commit message: Add files via upload
Changed lines of the file:
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@@
     )
   )
-  (global_label "12V_out" (shape input) (at 173.99 119.38 0) (fields_autoplaced)
+  (global_label "GND12V" (shape input) (at 173.99 119.38 0) (fields_autoplaced)
     (effects (font (size 1.27 1.27)) (justify left))
-    (property "Intersheet References" "${INTERSHEET_REFS}" (id 0) (at 183.9021 119.3006 0)
-      (effects (font (size 1.27 1.27)) (justify left) hide)
-    )
-  )
-  (global_label "5V_out" (shape input) (at 152.4 180.34 0) (fields_autoplaced)
+    (property "Intersheet References" "${INTERSHEET_REFS}" (id 0) (at 183.7812 119.3006 0)
+      (effects (font (size 1.27 1.27)) (justify left) hide)
+    )
+  )
+  (global_label "GND5V" (shape input) (at 152.4 180.34 0) (fields_autoplaced)
     (effects (font (size 1.27 1.27)) (justify left))
-    (property "Intersheet References" "${INTERSHEET_REFS}" (id 0) (at 161.1026 180.2606 0)
+    (property "Intersheet References" "${INTERSHEET_REFS}" (id 0) (at 160.9817 180.2606 0)
       (effects (font (size 1.27 1.27)) (justify left) hide)
     )
@@
     )
   )
-  (global_label "3.3V_out" (shape input) (at 185.42 58.42 0) (fields_autoplaced)
+  (global_label "GND3.3V" (shape input) (at 185.42 58.42 0) (fields_autoplaced)
     (effects (font (size 1.27 1.27)) (justify left))
-    (property "Intersheet References" "${INTERSHEET_REFS}" (id 0) (at 195.9369 58.3406 0)
+    (property "Intersheet References" "${INTERSHEET_REFS}" (id 0) (at 195.816 58.3406 0)
       (effects (font (size 1.27 1.27)) (justify left) hide)
     )
@@
     )
     (pin "1")
-    (pin "5")
     (pin "2")
     (pin "3")
     (pin "4")
+    (pin "5")
     (pin "6")
   )

Commit message: Add files via upload
Parts:
- added J1: Screw_Terminal_01x02, TerminalBlock_MetzConnect:TerminalBlock_MetzConnect_Type055_RT01502HDWU_1x02_P5.00mm_Horizontal, symbol Connector:Screw_Terminal_01x02
- gave numbers to parts that had none: 1
- renumbered C6 to C31, R8 to R10
Connections:
- net +BATT: now also J1.1 (Pin_1)
- net -BATT: now also J1.2 (Pin_2)
