File: EECD-22-7/power.kicad_sch (KiCad schematic)
At the start: 29 parts, among them J1 Screw_Terminal_01x02, Q1 IRF6616, Q2 IRF6616, U3 LMR54406DBVR, U4 LMR54406DBVR, U5 LMR54406DBVR

Commit message: Add files via upload
Parts:
- L1: renamed from L3; value 12uH -> 12uH 100mR 1.6A
- U7: renamed from U5; footprint (none) -> LMR:lmr
- U8: renamed from U4; footprint (none) -> LMR:lmr
- U9: renamed from U3; footprint (none) -> LMR:lmr
- renumbered C9 to C10, C10 to C11, C7 to C12, C8 to C13, C6 to C14, C31 to C15, C4 to C16, C5 to C17, C13 to C6, C14 to C7, C11 to C8, C12 to C9, J1 to J3, L1 to L3, R5 to R10, R24 to R11, R10 to R4, R9 to R5, R7 to R6, R8 to R7, R20 to R8, R4 to R9

Commit message: Add files via upload
Parts:
- C10, C14, C6: value 100nF -> 100nF 1mR
- C11, C16, C8: value 10uF -> 10uF 4.5mR
- C12: value 10uF -> 10uF 20mR
- C13, C9: value 100nF -> 100nF 3mR
- C15: value 10uF -> 10uF 2.2mR
- C17: value 100nF -> 100nF 20mR
- C7: value 10uF -> 10uF 4.5 mR
- L2: value 15uH -> 15uH 90mR 1.6A
- L3: value 150uH -> 150uH 90mR 1.8A
Other:
- moved on the sheet: C12, C8
Changed lines of the file:
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@@
+    (stroke (width 0) (type default) (color 0 0 0 0))
+  )
+  (wire (pts (xy 80.01 40.64) (xy 80.01 39.37))
     (stroke (width 0) (type default) (color 0 0 0 0))
   )
@@
     (stroke (width 0) (type default) (color 0 0 0 0))
   )
-  (wire (pts (xy 80.01 58.42) (xy 80.01 52.07))
+  (wire (pts (xy 80.01 58.42) (xy 80.01 53.34))
     (stroke (width 0) (type default) (color 0 0 0 0))
   )
@@
     (stroke (width 0) (type default) (color 0 0 0 0))
   )
-  (wire (pts (xy 44.45 119.38) (xy 44.45 113.03))
+  (wire (pts (xy 44.45 119.38) (xy 44.45 114.3))
     (stroke (width 0) (type default) (color 0 0 0 0))
   )
@@
   )
   (wire (pts (xy 26.67 180.34) (xy 46.99 180.34))
+    (stroke (width 0) (type default) (color 0 0 0 0))
+  )
+  (wire (pts (xy 44.45 101.6) (xy 44.45 100.33))
     (stroke (width 0) (type default) (color 0 0 0 0))
   )
@@
     (in_bom yes) (on_board yes) (fields_autoplaced)
     (property "Reference" "L2" (id 0) (at 142.24 80.01 90))
-    (property "Value" "15uH" (id 1) (at 142.24 82.55 90))
+    (property "Value" "15uH 90mR 1.6A" (id 1) (at 142.24 82.55 90))
     (property "Footprint" "" (id 2) (at 142.24 86.36 0)
       (effects (font (size 1.27 1.27)) hide)
@@
       (effects (font (size 1.27 1.27)) (justify left))
     )
-    (property "Value" "100nF" (id 1) (at 64.77 107.9499 0)
+    (property "Value" "100nF 3mR" (id 1) (at 64.77 107.9499 0)
       (effects (font (size 1.27 1.27)) (justify left))
     )
@@
     (in_bom yes) (on_board yes) (fields_autoplaced)
     (property "Reference" "C10" (id 0) (at 119.38 77.47 90))
-    (property "Value" "100nF" (id 1) (at 119.38 80.01 90))
+    (property "Value" "100nF 1mR" (id 1) (at 119.38 80.01 90))
     (property "Footprint" "" (id 2) (at 119.38 86.36 0)
       (effects (font (size 1.27 1.27)) hide)
@@
   )
   (symbol (lib_id "Device:R") (at 85.09 180.34 270) (mirror x) (unit 1)
-    (in_bom yes) (on_board yes) (fields_autoplaced)
-    (property "Reference" "R11" (id 0) (at 85.09 173.99 90))
-    (property "Value" "10kR" (id 1) (at 85.09 176.53 90))
+    (in_bom yes) (on_board yes)
+    (property "Reference" "R11" (id 0) (at 82.55 175.26 90))
+    (property "Value" "10kR" (id 1) (at 82.55 177.8 90))
     (property "Footprint" "" (id 2) (at 85.09 182.118 90)
       (effects (font (size 1.27 1.27)) hide)
@@
     (pin "1")
   )
-  (symbol (lib_id "pspice:C") (at 80.01 45.72 0) (unit 1)
-    (in_bom yes) (on_board yes) (fields_autoplaced)
-    (property "Reference" "C8" (id 0) (at 85.09 44.4499 0)
-      (effects (font (size 1.27 1.27)) (justify left))
-    )
-    (property "Value" "10uF" (id 1) (at 85.09 46.9899 0)
-      (effects (font (size 1.27 1.27)) (justify left))
-    )
-    (property "Footprint" "" (id 2) (at 80.01 45.72 0)
-      (effects (font (size 1.27 1.27)) hide)
-    )
-    (property "Datasheet" "~" (id 3) (at 80.01 45.72 0)
+  (symbol (lib_id "pspice:C") (at 80.01 46.99 0) (unit 1)
+    (in_bom yes) (on_board yes)
+    (property "Reference" "C8" (id 0) (at 85.09 45.7199 0)
+      (effects (font (size 1.27 1.27)) (justify left))
+    )
+    (property "Value" "10uF 4.5mR" (id 1) (at 74.93 53.34 0)
+      (effects (font (size 1.27 1.27)) (justify left))
+    )
+    (property "Footprint" "" (id 2) (at 80.01 46.99 0)
+      (effects (font (size 1.27 1.27)) hide)
+    )
+    (property "Datasheet" "~" (id 3) (at 80.01 46.99 0)
       (effects (font (size 1.27 1.27)) hide)
     )
@@
     (in_bom yes) (on_board yes) (fields_autoplaced)
     (property "Reference" "C14" (id 0) (at 97.79 138.43 90))
-    (property "Value" "100nF" (id 1) (at 97.79 140.97 90))
+    (property "Value" "100nF 1mR" (id 1) (at 97.79 140.97 90))
     (property "Footprint" "" (id 2) (at 97.79 147.32 0)
       (effects (font (size 1.27 1.27)) hide)
@@
   )
   (symbol (lib_id "pspice:C") (at 46.99 167.64 0) (unit 1)
-    (in_bom yes) (on_board yes) (fields_autoplaced)
+    (in_bom yes) (on_board yes)
     (property "Reference" "C16" (id 0) (at 52.07 166.3699 0)
       (effects (font (size 1.27 1.27)) (justify left))
     )
-    (property "Value" "10uF" (id 1) (at 52.07 168.9099 0)
+    (property "Value" "10uF 4.5mR" (id 1) (at 41.91 175.26 0)
       (effects (font (size 1.27 1.27)) (justify left))
     )
@@
     (pin "1")
   )
-  (symbol (lib_id "pspice:C") (at 44.45 106.68 0) (unit 1)
-    (in_bom yes) (on_board yes) (fields_autoplaced)
-    (property "Reference" "C12" (id 0) (at 49.53 105.4099 0)
-      (effects (font (size 1.27 1.27)) (justify left))
-    )
-    (property "Value" "10uF" (id 1) (at 49.53 107.9499 0)
-      (effects (font (size 1.27 1.27)) (justify left))
-    )
-    (property "Footprint" "" (id 2) (at 44.45 106.68 0)
-      (effects (font (size 1.27 1.27)) hide)
-    )
-    (property "Datasheet" "~" (id 3) (at 44.45 106.68 0)
+  (symbol (lib_id "pspice:C") (at 44.45 107.95 0) (unit 1)
+    (in_bom yes) (on_board yes)
+    (property "Reference" "C12" (id 0) (at 49.53 106.6799 0)
+      (effects (font (size 1.27 1.27)) (justify left))
+    )
+    (property "Value" "10uF 20mR" (id 1) (at 39.37 115.57 0)
+      (effects (font (size 1.27 1.27)) (justify left))
+    )
+    (property "Footprint" "" (id 2) (at 44.45 107.95 0)
+      (effects (font (size 1.27 1.27)) hide)
+    )
+    (property "Datasheet" "~" (id 3) (at 44.45 107.95 0)
       (effects (font (size 1.27 1.27)) hide)
     )
@@
       (effects (font (size 1.27 1.27)) (justify left))
     )
-    (property "Value" "10uF" (id 1) (at 171.45 104.1399 0)
+    (property "Value" "10uF 4.5mR" (id 1) (at 171.45 104.1399 0)
       (effects (font (size 1.27 1.27)) (justify left))
     )
@@
       (effects (font (size 1.27 1.27)) (justify left))
     )
-    (property "Value" "10uF" (id 1) (at 149.86 165.0999 0)
+    (property "Value" "10uF 2.2mR" (id 1) (at 149.86 165.0999 0)
       (effects (font (size 1.27 1.27)) (justify left))
     )
@@
   )
   (symbol (lib_id "pspice:C") (at 95.25 45.72 0) (unit 1)
-    (in_bom yes) (on_board yes) (fields_autoplaced)
+    (in_bom yes) (on_board yes)
     (property "Reference" "C9" (id 0) (at 100.33 44.4499 0)
       (effects (font (size 1.27 1.27)) (justify left))
     )
-    (property "Value" "100nF" (id 1) (at 100.33 46.9899 0)
+    (property "Value" "100nF 3mR" (id 1) (at 96.52 50.8 0)
       (effects (font (size 1.27 1.27)) (justify left))
     )
@@
     (in_bom yes) (on_board yes) (fields_autoplaced)
     (property "Reference" "L3" (id 0) (at 120.65 140.97 90))
-    (property "Value" "150uH" (id 1) (at 120.65 143.51 90))
+    (property "Value" "150uH 90mR 1.8A" (id 1) (at 120.65 143.51 90))
     (property "Footprint" "" (id 2) (at 120.65 147.32 0)
       (effects (font (size 1.27 1.27)) hide)
@@
     (in_bom yes) (on_board yes) (fields_autoplaced)
     (property "Reference" "C6" (id 0) (at 130.81 16.51 90))
-    (property "Value" "100nF" (id 1) (at 130.81 19.05 90))
+    (property "Value" "100nF 1mR" (id 1) (at 130.81 19.05 90))
     (property "Footprint" "" (id 2) (at 130.81 25.4 0)
       (effects (font (size 1.27 1.27)) hide)
@@
       (effects (font (size 1.27 1.27)) (justify left))
     )
-    (property "Value" "10uF" (id 1) (at 182.88 43.1799 0)
+    (property "Value" "10uF 4.5 mR" (id 1) (at 182.88 43.1799 0)
       (effects (font (size 1.27 1.27)) (justify left))
     )
@@
   )
   (symbol (lib_id "pspice:C") (at 62.23 167.64 0) (unit 1)
-    (in_bom yes) (on_board yes) (fields_autoplaced)
+    (in_bom yes) (on_board yes)
     (property "Reference" "C17" (id 0) (at 67.31 166.3699 0)
       (effects (font (size 1.27 1.27)) (justify left))
     )
-    (property "Value" "100nF" (id 1) (at 67.31 168.9099 0)
-      (effects (font (size 1.27 1.27)) (justify left))
-    )
+    (property "Value" "100nF 20mR" (id 1) (at 63.5 172.72 0)
+      (effects (font (size 1.27 1.27)) (justify left))
+    )

Commit message: Add files via upload
Parts:
- L1: footprint (none) -> inductor:NPI54C120MTRF
- L2: footprint (none) -> inductor:NPI75C150MTRF
- L3: value 150uH 90mR 1.8A -> 15uH 90mR 1.8A; footprint (none) -> inductor:NPI75C150MTRF
Changed lines of the file:
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@@
     (property "Reference" "L2" (id 0) (at 142.24 80.01 90))
     (property "Value" "15uH 90mR 1.6A" (id 1) (at 142.24 82.55 90))
-    (property "Footprint" "" (id 2) (at 142.24 86.36 0)
+    (property "Footprint" "inductor:NPI75C150MTRF" (id 2) (at 142.24 86.36 0)
       (effects (font (size 1.27 1.27)) hide)
     )
@@
     (property "Reference" "L1" (id 0) (at 153.67 19.05 90))
     (property "Value" "12uH 100mR 1.6A" (id 1) (at 153.67 21.59 90))
-    (property "Footprint" "" (id 2) (at 153.67 25.4 0)
+    (property "Footprint" "inductor:NPI54C120MTRF" (id 2) (at 153.67 25.4 0)
       (effects (font (size 1.27 1.27)) hide)
     )
@@
     (in_bom yes) (on_board yes) (fields_autoplaced)
     (property "Reference" "L3" (id 0) (at 120.65 140.97 90))
-    (property "Value" "150uH 90mR 1.8A" (id 1) (at 120.65 143.51 90))
-    (property "Footprint" "" (id 2) (at 120.65 147.32 0)
-      (effects (font (size 1.27 1.27)) hide)
-    )
+    (property "Value" "15uH 90mR 1.8A" (id 1) (at 120.65 143.51 90))
+    (property "Footprint" "inductor:NPI75C150MTRF" (id 2) (at 120.65 147.32 0)
+      (effects (font (size 1.27 1.27)) hide)
+    )

Commit message: Add files via upload
Changed lines of the file:
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@@
     (pin "3")
-  )
-  (symbol (lib_id "power:PWR_FLAG") (at 273.05 154.94 180) (unit 1)
-    (in_bom yes) (on_board yes) (fields_autoplaced)
-    (property "Reference" "#FLG05" (id 0) (at 273.05 156.845 0)
-      (effects (font (size 1.27 1.27)) hide)
-    )
-    (property "Value" "PWR_FLAG" (id 1) (at 273.05 160.02 0))
-    (property "Footprint" "" (id 2) (at 273.05 154.94 0)
-      (effects (font (size 1.27 1.27)) hide)
-    )
-    (property "Datasheet" "~" (id 3) (at 273.05 154.94 0)
-      (effects (font (size 1.27 1.27)) hide)
-    )
-    (pin "1")
   )
   (symbol (lib_id "power:GND") (at 106.68 58.42 0) (unit 1)
@@
       (effects (font (size 1.27 1.27)) hide)
     )
-    (pin "1")
-  )
-  (symbol (lib_id "power:-BATT") (at 273.05 154.94 0) (unit 1)
-    (in_bom yes) (on_board yes) (fields_autoplaced)
-    (property "Reference" "#PWR016" (id 0) (at 273.05 158.75 0)
-      (effects (font (size 1.27 1.27)) hide)
-    )
-    (property "Value" "-BATT" (id 1) (at 275.59 153.6699 0)
-      (effects (font (size 1.27 1.27)) (justify left))
-    )
-    (property "Footprint" "" (id 2) (at 273.05 154.94 0)
-      (effects (font (size 1.27 1.27)) hide)
-    )
-    (property "Datasheet" "" (id 3) (at 273.05 154.94 0)
-      (effects (font (size 1.27 1.27)) hide)
-    )

Commit message: Add files via upload
Parts:
- C10, C11, C12, C13, C14, C15, C16, C17, C6, C7, C8, C9: footprint (none) -> Capacitor_SMD:C_0603_1608Metric
- R10, R11, R4, R5, R6, R7, R8, R9: footprint (none) -> Resistor_SMD:R_0603_1608Metric
Changed lines of the file:
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@@
       (effects (font (size 1.27 1.27)) (justify left))
     )
-    (property "Footprint" "" (id 2) (at 59.69 106.68 0)
+    (property "Footprint" "Capacitor_SMD:C_0603_1608Metric" (id 2) (at 59.69 106.68 0)
       (effects (font (size 1.27 1.27)) hide)
     )
@@
     (property "Reference" "C10" (id 0) (at 119.38 77.47 90))
     (property "Value" "100nF 1mR" (id 1) (at 119.38 80.01 90))
-    (property "Footprint" "" (id 2) (at 119.38 86.36 0)
+    (property "Footprint" "Capacitor_SMD:C_0603_1608Metric" (id 2) (at 119.38 86.36 0)
       (effects (font (size 1.27 1.27)) hide)
     )
@@
     (property "Reference" "R11" (id 0) (at 82.55 175.26 90))
     (property "Value" "10kR" (id 1) (at 82.55 177.8 90))
-    (property "Footprint" "" (id 2) (at 85.09 182.118 90)
+    (property "Footprint" "Resistor_SMD:R_0603_1608Metric" (id 2) (at 85.09 182.118 90)
       (effects (font (size 1.27 1.27)) hide)
     )
@@
       (effects (font (size 1.27 1.27)) (justify left))
     )
-    (property "Footprint" "" (id 2) (at 148.082 113.03 90)
+    (property "Footprint" "Resistor_SMD:R_0603_1608Metric" (id 2) (at 148.082 113.03 90)
       (effects (font (size 1.27 1.27)) hide)
     )
@@
       (effects (font (size 1.27 1.27)) (justify left))
     )
-    (property "Footprint" "" (id 2) (at 159.512 34.29 90)
+    (property "Footprint" "Resistor_SMD:R_0603_1608Metric" (id 2) (at 159.512 34.29 90)
       (effects (font (size 1.27 1.27)) hide)
     )
@@
       (effects (font (size 1.27 1.27)) (justify left))
     )
-    (property "Footprint" "" (id 2) (at 80.01 46.99 0)
+    (property "Footprint" "Capacitor_SMD:C_0603_1608Metric" (id 2) (at 80.01 46.99 0)
       (effects (font (size 1.27 1.27)) hide)
     )
@@
     (property "Reference" "C14" (id 0) (at 97.79 138.43 90))
     (property "Value" "100nF 1mR" (id 1) (at 97.79 140.97 90))
-    (property "Footprint" "" (id 2) (at 97.79 147.32 0)
+    (property "Footprint" "Capacitor_SMD:C_0603_1608Metric" (id 2) (at 97.79 147.32 0)
       (effects (font (size 1.27 1.27)) hide)
     )
@@
       (effects (font (size 1.27 1.27)) (justify left))
     )
-    (property "Footprint" "" (id 2) (at 46.99 167.64 0)
+    (property "Footprint" "Capacitor_SMD:C_0603_1608Metric" (id 2) (at 46.99 167.64 0)
       (effects (font (size 1.27 1.27)) hide)
     )
@@
       (effects (font (size 1.27 1.27)) (justify left))
     )
-    (property "Footprint" "" (id 2) (at 44.45 107.95 0)
+    (property "Footprint" "Capacitor_SMD:C_0603_1608Metric" (id 2) (at 44.45 107.95 0)
       (effects (font (size 1.27 1.27)) hide)
     )
@@
       (effects (font (size 1.27 1.27)) (justify left))
     )
-    (property "Footprint" "" (id 2) (at 166.37 102.87 0)
+    (property "Footprint" "Capacitor_SMD:C_0603_1608Metric" (id 2) (at 166.37 102.87 0)
       (effects (font (size 1.27 1.27)) hide)
     )
@@
       (effects (font (size 1.27 1.27)) (justify left))
     )
-    (property "Footprint" "" (id 2) (at 144.78 163.83 0)
+    (property "Footprint" "Capacitor_SMD:C_0603_1608Metric" (id 2) (at 144.78 163.83 0)
       (effects (font (size 1.27 1.27)) hide)
     )
@@
       (effects (font (size 1.27 1.27)) (justify left))
     )
-    (property "Footprint" "" (id 2) (at 95.25 45.72 0)
+    (property "Footprint" "Capacitor_SMD:C_0603_1608Metric" (id 2) (at 95.25 45.72 0)
       (effects (font (size 1.27 1.27)) hide)
     )
@@
     (property "Reference" "C6" (id 0) (at 130.81 16.51 90))
     (property "Value" "100nF 1mR" (id 1) (at 130.81 19.05 90))
-    (property "Footprint" "" (id 2) (at 130.81 25.4 0)
+    (property "Footprint" "Capacitor_SMD:C_0603_1608Metric" (id 2) (at 130.81 25.4 0)
       (effects (font (size 1.27 1.27)) hide)
     )
@@
       (effects (font (size 1.27 1.27)) (justify left))
     )
-    (property "Footprint" "" (id 2) (at 148.082 95.25 90)
+    (property "Footprint" "Resistor_SMD:R_0603_1608Metric" (id 2) (at 148.082 95.25 90)
       (effects (font (size 1.27 1.27)) hide)
     )
@@
       (effects (font (size 1.27 1.27)) (justify left))
     )
-    (property "Footprint" "" (id 2) (at 126.492 156.21 90)
+    (property "Footprint" "Resistor_SMD:R_0603_1608Metric" (id 2) (at 126.492 156.21 90)
       (effects (font (size 1.27 1.27)) hide)
     )
@@
       (effects (font (size 1.27 1.27)) (justify left))
     )
-    (property "Footprint" "" (id 2) (at 177.8 41.91 0)
+    (property "Footprint" "Capacitor_SMD:C_0603_1608Metric" (id 2) (at 177.8 41.91 0)
       (effects (font (size 1.27 1.27)) hide)
     )
@@
       (effects (font (size 1.27 1.27)) (justify left))
     )
-    (property "Footprint" "" (id 2) (at 159.512 52.07 90)
+    (property "Footprint" "Resistor_SMD:R_0603_1608Metric" (id 2) (at 159.512 52.07 90)
       (effects (font (size 1.27 1.27)) hide)
     )
@@
     (property "Reference" "R8" (id 0) (at 77.47 113.03 90))
     (property "Value" "10kR" (id 1) (at 77.47 115.57 90))
-    (property "Footprint" "" (id 2) (at 77.47 121.158 90)
+    (property "Footprint" "Resistor_SMD:R_0603_1608Metric" (id 2) (at 77.47 121.158 90)
       (effects (font (size 1.27 1.27)) hide)
     )
@@
       (effects (font (size 1.27 1.27)) (justify left))
     )
-    (property "Footprint" "" (id 2) (at 62.23 167.64 0)
+    (property "Footprint" "Capacitor_SMD:C_0603_1608Metric" (id 2) (at 62.23 167.64 0)
       (effects (font (size 1.27 1.27)) hide)
     )
@@
       (effects (font (size 1.27 1.27)) (justify left))
     )
-    (property "Footprint" "" (id 2) (at 126.492 173.99 90)
-      (effects (font (size 1.27 1.27)) hide)
-    )
+    (property "Footprint" "Resistor_SMD:R_0603_1608Metric" (id 2) (at 126.492 173.99 90)
+      (effects (font (size 1.27 1.27)) hide)
+    )
