File: EECD-22-7/EECD-22-7.kicad_sch (KiCad schematic)
At the start: 3 parts, among them J1_I2C_Gamma_Sensor Conn_01x06_Female, U1_Pressure_Sensor MS5525DSO, U2_Temperature_Sensor TMP1075D

Commit message: Add files via upload
Other:
- added sheet measurements (measurements_sch.kicad_sch)
Changed lines of the file:
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@@
     (pin "6")
+  )
+  (sheet (at 15.24 242.57) (size 284.48 111.76) (fields_autoplaced)
+    (stroke (width 0.1524) (type solid) (color 0 0 0 0))
+    (fill (color 0 0 0 0.0000))
+    (property "Sheet name" "measurements" (id 0) (at 15.24 241.8584 0)
+      (effects (font (size 1.27 1.27)) (justify left bottom))
+    )
+    (property "Sheet file" "measurements_sch.kicad_sch" (id 1) (at 15.24 354.9146 0)
+      (effects (font (size 1.27 1.27)) (justify left top))
+    )
   )
   (sheet_instances
     (path "/" (page "1"))
+    (path "/6fbcc029-2e97-4cbb-aefe-dadd6dac0b49" (page "2"))
   )
   (symbol_instances
@@
       (reference "U2_Temperature_Sensor") (unit 1) (value "TMP1075D") (footprint "Package_SO:SO-8_3.9x4.9mm_P1.27mm")
     )
+    (path "/6fbcc029-2e97-4cbb-aefe-dadd6dac0b49/c24eb077-6d4a-4ccd-bd1c-9ae5a44d9429"
+      (reference "U?") (unit 1) (value "519") (footprint "")
+    )
   )

Commit message: Add files via upload
Other:
- added sheet communication (ultrasound_sch.kicad_sch)
- added sheet power converters (power.kicad_sch)
Changed lines of the file:
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@@
     (pin "6")
+  )
+  (sheet (at 17.78 375.92) (size 281.94 81.28) (fields_autoplaced)
+    (stroke (width 0.1524) (type solid) (color 0 0 0 0))
+    (fill (color 0 0 0 0.0000))
+    (property "Sheet name" "communication" (id 0) (at 17.78 375.2084 0)
+      (effects (font (size 1.27 1.27)) (justify left bottom))
+    )
+    (property "Sheet file" "ultrasound_sch.kicad_sch" (id 1) (at 17.78 457.7846 0)
+      (effects (font (size 1.27 1.27)) (justify left top))
+    )
   )
   (sheet (at 15.24 242.57) (size 284.48 111.76) (fields_autoplaced)
@@
     )
   )
+  (sheet (at 320.04 7.62) (size 124.46 203.2) (fields_autoplaced)
+    (stroke (width 0.1524) (type solid) (color 0 0 0 0))
+    (fill (color 0 0 0 0.0000))
+    (property "Sheet name" "power converters" (id 0) (at 320.04 6.9084 0)
+      (effects (font (size 1.27 1.27)) (justify left bottom))
+    )
+    (property "Sheet file" "power.kicad_sch" (id 1) (at 320.04 211.4046 0)
+      (effects (font (size 1.27 1.27)) (justify left top))
+    )
+  )
   (sheet_instances
     (path "/" (page "1"))
     (path "/6fbcc029-2e97-4cbb-aefe-dadd6dac0b49" (page "2"))
+    (path "/03efad70-c9aa-48a1-8756-ad404298714a" (page "3"))
+    (path "/9c7af212-65f3-4d36-9a7c-51f47c138f55" (page "4"))
   )
   (symbol_instances
+    (path "/03efad70-c9aa-48a1-8756-ad404298714a/358c6983-81cf-4558-aacb-35d3a5f778c5"
+      (reference "#PWR?") (unit 1) (value "+1V0") (footprint "")
+    )
+    (path "/03efad70-c9aa-48a1-8756-ad404298714a/f0e9981e-f1ec-415d-b90b-438ddaa7c882"
+      (reference "#PWR?") (unit 1) (value "GND") (footprint "")
+    )
+    (path "/03efad70-c9aa-48a1-8756-ad404298714a/be22a395-60aa-4885-bf5e-173116540bc5"
+      (reference "BZ1") (unit 1) (value "Piezo") (footprint "")
+    )
+    (path "/03efad70-c9aa-48a1-8756-ad404298714a/6f354bec-17a3-4ebf-9b29-8e9e2afe0ee7"
+      (reference "C1") (unit 1) (value "0.1uF") (footprint "")
+    )
+    (path "/03efad70-c9aa-48a1-8756-ad404298714a/76127282-4a58-4150-afae-0beec97e3c40"
+      (reference "D1") (unit 1) (value "1N4004") (footprint "Diode_THT:D_DO-41_SOD81_P10.16mm_Horizontal")
+    )
+    (path "/03efad70-c9aa-48a1-8756-ad404298714a/29e69c9a-c4b2-49e9-92ce-3b7aff26f405"
+      (reference "D2") (unit 1) (value "1N4004") (footprint "Diode_THT:D_DO-41_SOD81_P10.16mm_Horizontal")
+    )
     (path "/ab6339dd-3fd4-470b-88ba-ed003ffd90e2"
       (reference "J1_I2C_Gamma_Sensor") (unit 1) (value "Conn_01x06_Female") (footprint "")
+    )
+    (path "/03efad70-c9aa-48a1-8756-ad404298714a/082c7dd8-d570-485a-8a8c-7516fa7ad208"
+      (reference "R1") (unit 1) (value "100R") (footprint "")
+    )
+    (path "/03efad70-c9aa-48a1-8756-ad404298714a/e310a78b-1c0b-4b8a-9cad-4befb515f038"
+      (reference "R2") (unit 1) (value "470k") (footprint "")
     )
     (path "/ab543afa-5bfb-444f-a849-bb48797521b2"
       (reference "U1_Pressure_Sensor") (unit 1) (value "MS5525DSO") (footprint "")
     )
+    (path "/9c7af212-65f3-4d36-9a7c-51f47c138f55/cf0de218-f97d-40c7-864e-2518980e3d53"
+      (reference "U2") (unit 1) (value "LM25183NGUR") (footprint "")
+    )
     (path "/660be7d2-1f7a-4768-99a1-b2cc3f121f43"
       (reference "U2_Temperature_Sensor") (unit 1) (value "TMP1075D") (footprint "Package_SO:SO-8_3.9x4.9mm_P1.27mm")
     )
+    (path "/9c7af212-65f3-4d36-9a7c-51f47c138f55/912c63c5-5df7-4dcf-8c39-15d6624f0cd7"
+      (reference "U3") (unit 1) (value "LM5181NGUR") (footprint "")
+    )
     (path "/6fbcc029-2e97-4cbb-aefe-dadd6dac0b49/c24eb077-6d4a-4ccd-bd1c-9ae5a44d9429"

Commit message: Add files via upload
Parts:
- removed J1_I2C_Gamma_Sensor: Conn_01x06_Female, symbol Connector:Conn_01x06_Female
- removed U1_Pressure_Sensor: MS5525DSO, symbol Sensor_Pressure:MS5525DSO
- removed U2_Temperature_Sensor: TMP1075D, Package_SO:SO-8_3.9x4.9mm_P1.27mm, symbol Sensor_Temperature:TMP1075D
Other:
- added sheet main (untitled.kicad_sch)
Changed lines of the file:
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@@
 (kicad_sch (version 20211123) (generator eeschema)
   (paper "A4")
-  (symbol (lib_id "Sensor_Temperature:TMP1075D") (at 178.943 109.22 0) (unit 1)
-    (in_bom yes) (on_board yes) (fields_autoplaced)
-    (property "Reference" "U2_Temperature_Sensor" (id 0) (at 180.9624 99.06 0)
-      (effects (font (size 1.27 1.27)) (justify left))
-    )
-    (property "Value" "TMP1075D" (id 1) (at 180.9624 101.6 0)
-      (effects (font (size 1.27 1.27)) (justify left))
-    )
-    (property "Footprint" "Package_SO:SO-8_3.9x4.9mm_P1.27mm" (id 2) (at 178.943 115.57 0)
-      (effects (font (size 1.27 1.27)) hide)
-    )
-    (property "Datasheet" "https://www.ti.com/lit/gpn/tmp1075" (id 3) (at 178.943 109.22 0)
-      (effects (font (size 1.27 1.27)) hide)
-    )
-    (pin "1")
-    (pin "2")
-    (pin "3")
-    (pin "4")
-    (pin "5")
-    (pin "6")
-    (pin "7")
-    (pin "8")
-  )
-  (symbol (lib_id "Sensor_Pressure:MS5525DSO") (at 183.515 74.676 0) (unit 1)
-    (in_bom yes) (on_board yes) (fields_autoplaced)
-    (property "Reference" "U1_Pressure_Sensor" (id 0) (at 185.5344 59.436 0)
-      (effects (font (size 1.27 1.27)) (justify left))
-    )
-    (property "Value" "MS5525DSO" (id 1) (at 185.5344 61.976 0)
-      (effects (font (size 1.27 1.27)) (justify left))
-    )
-    (property "Footprint" "" (id 2) (at 183.515 88.646 0)
-      (effects (font (size 1.27 1.27)) hide)
-    )
-    (property "Datasheet" "https://www.te.com/commerce/DocumentDelivery/DDEController?Action=srchrtrv&DocNm=MS5525DSO&DocType=DS&DocLang=English" (id 3) (at 183.515 91.186 0)
-      (effects (font (size 1.27 1.27)) hide)
-    )
-    (pin "1")
-    (pin "10")
-    (pin "11")
-    (pin "12")
-    (pin "13")
-    (pin "14")
-    (pin "2")
-    (pin "3")
-    (pin "4")
-    (pin "5")
-    (pin "6")
-    (pin "7")
-    (pin "8")
-    (pin "9")
-  )
-  (symbol (lib_id "Connector:Conn_01x06_Female") (at 82.931 115.316 0) (unit 1)
-    (in_bom yes) (on_board yes) (fields_autoplaced)
-    (property "Reference" "J1_I2C_Gamma_Sensor" (id 0) (at 83.82 115.3159 0)
-      (effects (font (size 1.27 1.27)) (justify left))
-    )
-    (property "Value" "Conn_01x06_Female" (id 1) (at 83.82 117.8559 0)
-      (effects (font (size 1.27 1.27)) (justify left))
-    )
-    (property "Footprint" "" (id 2) (at 82.931 115.316 0))
-    (property "Datasheet" "~" (id 3) (at 82.931 115.316 0)
-      (effects (font (size 1.27 1.27)) hide)
-    )
-    (pin "1")
-    (pin "2")
-    (pin "3")
-    (pin "4")
-    (pin "5")
-    (pin "6")
-  )
-  (sheet (at 17.78 375.92) (size 281.94 81.28) (fields_autoplaced)
+  (sheet (at 88.9 104.14) (size 38.1 36.83) (fields_autoplaced)
     (stroke (width 0.1524) (type solid) (color 0 0 0 0))
     (fill (color 0 0 0 0.0000))
-    (property "Sheet name" "communication" (id 0) (at 17.78 375.2084 0)
+    (property "Sheet name" "communication" (id 0) (at 88.9 103.4284 0)
       (effects (font (size 1.27 1.27)) (justify left bottom))
     )
-    (property "Sheet file" "ultrasound_sch.kicad_sch" (id 1) (at 17.78 457.7846 0)
+    (property "Sheet file" "ultrasound_sch.kicad_sch" (id 1) (at 88.9 141.5546 0)
       (effects (font (size 1.27 1.27)) (justify left top))
     )
   )
-  (sheet (at 15.24 242.57) (size 284.48 111.76) (fields_autoplaced)
+  (sheet (at 134.62 54.61) (size 39.37 39.37) (fields_autoplaced)
     (stroke (width 0.1524) (type solid) (color 0 0 0 0))
     (fill (color 0 0 0 0.0000))
-    (property "Sheet name" "measurements" (id 0) (at 15.24 241.8584 0)
+    (property "Sheet name" "measurements" (id 0) (at 134.62 53.8984 0)
       (effects (font (size 1.27 1.27)) (justify left bottom))
     )
-    (property "Sheet file" "measurements_sch.kicad_sch" (id 1) (at 15.24 354.9146 0)
+    (property "Sheet file" "measurements_sch.kicad_sch" (id 1) (at 134.62 94.5646 0)
       (effects (font (size 1.27 1.27)) (justify left top))
     )
   )
-  (sheet (at 320.04 7.62) (size 124.46 203.2) (fields_autoplaced)
+  (sheet (at 88.9 54.61) (size 38.1 39.37) (fields_autoplaced)
     (stroke (width 0.1524) (type solid) (color 0 0 0 0))
     (fill (color 0 0 0 0.0000))
-    (property "Sheet name" "power converters" (id 0) (at 320.04 6.9084 0)
+    (property "Sheet name" "main" (id 0) (at 88.9 53.8984 0)
       (effects (font (size 1.27 1.27)) (justify left bottom))
     )
-    (property "Sheet file" "power.kicad_sch" (id 1) (at 320.04 211.4046 0)
+    (property "Sheet file" "untitled.kicad_sch" (id 1) (at 88.9 94.5646 0)
+      (effects (font (size 1.27 1.27)) (justify left top))
+    )
+  )
+  (sheet (at 134.62 104.14) (size 38.1 36.83) (fields_autoplaced)
+    (stroke (width 0.1524) (type solid) (color 0 0 0 0))
+    (fill (color 0 0 0 0.0000))
+    (property "Sheet name" "power converters" (id 0) (at 134.62 103.4284 0)
+      (effects (font (size 1.27 1.27)) (justify left bottom))
+    )
+    (property "Sheet file" "power.kicad_sch" (id 1) (at 134.62 141.5546 0)
       (effects (font (size 1.27 1.27)) (justify left top))
     )
@@
     (path "/03efad70-c9aa-48a1-8756-ad404298714a" (page "3"))
     (path "/9c7af212-65f3-4d36-9a7c-51f47c138f55" (page "4"))
+    (path "/942d51a0-7498-4db1-b32e-613df6c3f987" (page "5"))
   )
   (symbol_instances
@@
       (reference "D2") (unit 1) (value "1N4004") (footprint "Diode_THT:D_DO-41_SOD81_P10.16mm_Horizontal")
     )
-    (path "/ab6339dd-3fd4-470b-88ba-ed003ffd90e2"
-      (reference "J1_I2C_Gamma_Sensor") (unit 1) (value "Conn_01x06_Female") (footprint "")
+    (path "/942d51a0-7498-4db1-b32e-613df6c3f987/eb7f4799-9c5b-4169-b632-4f576f2e8b1d"
+      (reference "J1_I2C_Gamma_Sensor?") (unit 1) (value "Conn_01x06_Female") (footprint "")
     )
     (path "/03efad70-c9aa-48a1-8756-ad404298714a/082c7dd8-d570-485a-8a8c-7516fa7ad208"
@@
       (reference "R2") (unit 1) (value "470k") (footprint "")
     )
-    (path "/ab543afa-5bfb-444f-a849-bb48797521b2"
-      (reference "U1_Pressure_Sensor") (unit 1) (value "MS5525DSO") (footprint "")
+    (path "/942d51a0-7498-4db1-b32e-613df6c3f987/adbee1bf-d88c-4783-a838-2c603551276b"
+      (reference "U1_Pressure_Sensor?") (unit 1) (value "MS5525DSO") (footprint "")
     )
     (path "/9c7af212-65f3-4d36-9a7c-51f47c138f55/cf0de218-f97d-40c7-864e-2518980e3d53"
       (reference "U2") (unit 1) (value "LM25183NGUR") (footprint "")
     )
-    (path "/660be7d2-1f7a-4768-99a1-b2cc3f121f43"
-      (reference "U2_Temperature_Sensor") (unit 1) (value "TMP1075D") (footprint "Package_SO:SO-8_3.9x4.9mm_P1.27mm")
+    (path "/942d51a0-7498-4db1-b32e-613df6c3f987/b777e41f-e4bb-4932-9d75-ce2dabd6efea"
+      (reference "U2_Temperature_Sensor?") (unit 1) (value "TMP1075D") (footprint "Package_SO:SO-8_3.9x4.9mm_P1.27mm")
     )
     (path "/9c7af212-65f3-4d36-9a7c-51f47c138f55/912c63c5-5df7-4dcf-8c39-15d6624f0cd7"

Commit message: Add files via upload
Other:
- added sheet mcu (mcu_sch.kicad_sch)
Changed lines of the file:
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@@
+    )
+  )
+  (sheet (at 177.8 54.61) (size 40.64 39.37) (fields_autoplaced)
+    (stroke (width 0.1524) (type solid) (color 0 0 0 0))
+    (fill (color 0 0 0 0.0000))
+    (property "Sheet name" "mcu" (id 0) (at 177.8 53.8984 0)
+      (effects (font (size 1.27 1.27)) (justify left bottom))
+    )
+    (property "Sheet file" "mcu_sch.kicad_sch" (id 1) (at 177.8 94.5646 0)
+      (effects (font (size 1.27 1.27)) (justify left top))
     )
   )
@@
     (path "/9c7af212-65f3-4d36-9a7c-51f47c138f55" (page "4"))
     (path "/942d51a0-7498-4db1-b32e-613df6c3f987" (page "5"))
+    (path "/415dd66c-310d-4150-9e33-ee8b65aef7bc" (page "6"))
   )
   (symbol_instances
@@
       (reference "U3") (unit 1) (value "LM5181NGUR") (footprint "")
     )
+    (path "/942d51a0-7498-4db1-b32e-613df6c3f987/a5acd85e-3114-4004-a4be-0df8305cfbf6"
+      (reference "U?") (unit 1) (value "MAX485E") (footprint "")
+    )
+    (path "/415dd66c-310d-4150-9e33-ee8b65aef7bc/b8e1c121-555c-4163-905a-781916653ef8"
+      (reference "U?") (unit 1) (value "ATmega644V-10M") (footprint "Package_DFN_QFN:QFN-44-1EP_7x7mm_P0.5mm_EP5.2x5.2mm")
+    )
     (path "/6fbcc029-2e97-4cbb-aefe-dadd6dac0b49/c24eb077-6d4a-4ccd-bd1c-9ae5a44d9429"

Commit message: Add files via upload
Other:
- removed sheet main
Changed lines of the file:
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@@
 (kicad_sch (version 20211123) (generator eeschema)
   (paper "A4")
-  (sheet (at 88.9 104.14) (size 38.1 36.83) (fields_autoplaced)
-    (stroke (width 0.1524) (type solid) (color 0 0 0 0))
-    (fill (color 0 0 0 0.0000))
-    (property "Sheet name" "communication" (id 0) (at 88.9 103.4284 0)
-      (effects (font (size 1.27 1.27)) (justify left bottom))
-    )
-    (property "Sheet file" "ultrasound_sch.kicad_sch" (id 1) (at 88.9 141.5546 0)
-      (effects (font (size 1.27 1.27)) (justify left top))
-    )
-  )
-  (sheet (at 177.8 54.61) (size 40.64 39.37) (fields_autoplaced)
-    (stroke (width 0.1524) (type solid) (color 0 0 0 0))
-    (fill (color 0 0 0 0.0000))
-    (property "Sheet name" "mcu" (id 0) (at 177.8 53.8984 0)
-      (effects (font (size 1.27 1.27)) (justify left bottom))
-    )
-    (property "Sheet file" "mcu_sch.kicad_sch" (id 1) (at 177.8 94.5646 0)
-      (effects (font (size 1.27 1.27)) (justify left top))
-    )
-  )
-  (sheet (at 134.62 54.61) (size 39.37 39.37) (fields_autoplaced)
+  (sheet (at 59.69 104.14) (size 67.31 36.83) (fields_autoplaced)
+    (stroke (width 0.1524) (type solid) (color 0 0 0 0))
+    (fill (color 0 0 0 0.0000))
+    (property "Sheet name" "communication" (id 0) (at 59.69 103.4284 0)
+      (effects (font (size 1.27 1.27)) (justify left bottom))
+    )
+    (property "Sheet file" "ultrasound_sch.kicad_sch" (id 1) (at 59.69 141.5546 0)
+      (effects (font (size 1.27 1.27)) (justify left top))
+    )
+  )
+  (sheet (at 59.69 54.61) (size 67.31 39.37) (fields_autoplaced)
+    (stroke (width 0.1524) (type solid) (color 0 0 0 0))
+    (fill (color 0 0 0 0.0000))
+    (property "Sheet name" "mcu" (id 0) (at 59.69 53.8984 0)
+      (effects (font (size 1.27 1.27)) (justify left bottom))
+    )
+    (property "Sheet file" "mcu_sch.kicad_sch" (id 1) (at 59.69 94.5646 0)
+      (effects (font (size 1.27 1.27)) (justify left top))
+    )
+  )
+  (sheet (at 134.62 54.61) (size 71.12 39.37) (fields_autoplaced)
     (stroke (width 0.1524) (type solid) (color 0 0 0 0))
     (fill (color 0 0 0 0.0000))
@@
     )
   )
-  (sheet (at 88.9 54.61) (size 38.1 39.37) (fields_autoplaced)
-    (stroke (width 0.1524) (type solid) (color 0 0 0 0))
-    (fill (color 0 0 0 0.0000))
-    (property "Sheet name" "main" (id 0) (at 88.9 53.8984 0)
-      (effects (font (size 1.27 1.27)) (justify left bottom))
-    )
-    (property "Sheet file" "untitled.kicad_sch" (id 1) (at 88.9 94.5646 0)
-      (effects (font (size 1.27 1.27)) (justify left top))
-    )
-  )
-  (sheet (at 134.62 104.14) (size 38.1 36.83) (fields_autoplaced)
+  (sheet (at 134.62 104.14) (size 69.85 36.83) (fields_autoplaced)
     (stroke (width 0.1524) (type solid) (color 0 0 0 0))
     (fill (color 0 0 0 0.0000))
@@
     (path "/03efad70-c9aa-48a1-8756-ad404298714a" (page "3"))
     (path "/9c7af212-65f3-4d36-9a7c-51f47c138f55" (page "4"))
-    (path "/942d51a0-7498-4db1-b32e-613df6c3f987" (page "5"))
     (path "/415dd66c-310d-4150-9e33-ee8b65aef7bc" (page "6"))
   )
@@
       (reference "C14") (unit 1) (value "10uF") (footprint "")
     )
+    (path "/415dd66c-310d-4150-9e33-ee8b65aef7bc/1c4d9d80-004c-4aae-a0ee-6724f8a616e3"
+      (reference "C15") (unit 1) (value "100nF") (footprint "")
+    )
+    (path "/415dd66c-310d-4150-9e33-ee8b65aef7bc/972e407f-d96f-4fe1-829a-f637cec60c2d"
+      (reference "C16") (unit 1) (value "100nF") (footprint "")
+    )
+    (path "/415dd66c-310d-4150-9e33-ee8b65aef7bc/e764f57b-450b-4c5b-bf87-8a19fecd14a8"
+      (reference "C17") (unit 1) (value "100nF") (footprint "")
+    )
+    (path "/415dd66c-310d-4150-9e33-ee8b65aef7bc/be80ec3b-a7a3-49a5-bd46-b636724fff6b"
+      (reference "C18") (unit 1) (value "10uF") (footprint "")
+    )
+    (path "/415dd66c-310d-4150-9e33-ee8b65aef7bc/894a4b68-d98b-4c78-96f1-229c7ecfff98"
+      (reference "C19") (unit 1) (value "100nF") (footprint "")
+    )
+    (path "/415dd66c-310d-4150-9e33-ee8b65aef7bc/6a116c90-fb0f-4a52-bb29-c9efba039654"
+      (reference "C20") (unit 1) (value "1uF") (footprint "")
+    )
     (path "/03efad70-c9aa-48a1-8756-ad404298714a/76127282-4a58-4150-afae-0beec97e3c40"
       (reference "D1") (unit 1) (value "1N4004") (footprint "Diode_THT:D_DO-41_SOD81_P10.16mm_Horizontal")
@@
       (reference "D2") (unit 1) (value "1N4004") (footprint "Diode_THT:D_DO-41_SOD81_P10.16mm_Horizontal")
     )
-    (path "/942d51a0-7498-4db1-b32e-613df6c3f987/eb7f4799-9c5b-4169-b632-4f576f2e8b1d"
+    (path "/6fbcc029-2e97-4cbb-aefe-dadd6dac0b49/23c26929-da1f-4eb3-a538-739afcee9733"
       (reference "J1_I2C_Gamma_Sensor?") (unit 1) (value "Conn_01x06_Female") (footprint "")
     )
@@
       (reference "L3") (unit 1) (value "12uH") (footprint "")
     )
+    (path "/9c7af212-65f3-4d36-9a7c-51f47c138f55/3bc44259-c6f5-47cb-bbbc-e193a255103d"
+      (reference "Q1") (unit 1) (value "IRF6616") (footprint "Package_DirectFET:DirectFET_MX")
+    )
+    (path "/9c7af212-65f3-4d36-9a7c-51f47c138f55/12a8aca8-2257-4379-90ff-647554e3744d"
+      (reference "Q2") (unit 1) (value "IRF6616") (footprint "Package_DirectFET:DirectFET_MX")
+    )
     (path "/03efad70-c9aa-48a1-8756-ad404298714a/082c7dd8-d570-485a-8a8c-7516fa7ad208"
       (reference "R1") (unit 1) (value "100R") (footprint "")
@@
       (reference "R9") (unit 1) (value "22kR") (footprint "")
     )
+    (path "/415dd66c-310d-4150-9e33-ee8b65aef7bc/b8f2ff96-ccec-46c9-a0e8-af4385b84d4f"
+      (reference "R15") (unit 1) (value "10kR") (footprint "")
+    )
+    (path "/415dd66c-310d-4150-9e33-ee8b65aef7bc/38ed9b93-44f8-48f9-ae47-04c489933495"
+      (reference "R16") (unit 1) (value "500kR") (footprint "")
+    )
+    (path "/9c7af212-65f3-4d36-9a7c-51f47c138f55/db0e37c9-c715-4c6d-bef2-8e9b8028a567"
+      (reference "R20") (unit 1) (value "10kR") (footprint "")
+    )
+    (path "/9c7af212-65f3-4d36-9a7c-51f47c138f55/3c5dfd03-89d6-4be0-9a92-9c429350514d"
+      (reference "R?") (unit 1) (value "10kR") (footprint "")
+    )
+    (path "/415dd66c-310d-4150-9e33-ee8b65aef7bc/4a7379e1-ac0a-4ddc-88a3-fd1e1ca6e517"
+      (reference "SW1") (unit 1) (value "SW_Push") (footprint "")
+    )
     (path "/415dd66c-310d-4150-9e33-ee8b65aef7bc/03e88226-cd4c-495e-8240-f30f511ef3fc"
       (reference "U1") (unit 1) (value "STM32F103CBUx") (footprint "Package_DFN_QFN:QFN-48-1EP_7x7mm_P0.5mm_EP5.6x5.6mm")
     )
-    (path "/942d51a0-7498-4db1-b32e-613df6c3f987/adbee1bf-d88c-4783-a838-2c603551276b"
+    (path "/6fbcc029-2e97-4cbb-aefe-dadd6dac0b49/9d586274-0455-46fc-85aa-d0245b458ee2"
       (reference "U1_Pressure_Sensor?") (unit 1) (value "MS5525DSO") (footprint "")
     )
-    (path "/942d51a0-7498-4db1-b32e-613df6c3f987/b777e41f-e4bb-4932-9d75-ce2dabd6efea"
+    (path "/6fbcc029-2e97-4cbb-aefe-dadd6dac0b49/5e9a6694-3a90-4221-9a42-ceda3055f854"
       (reference "U2_Temperature_Sensor?") (unit 1) (value "TMP1075D") (footprint "Package_SO:SO-8_3.9x4.9mm_P1.27mm")
     )
@@
       (reference "U5") (unit 1) (value "LMR54406DBVR") (footprint "")
     )
-    (path "/942d51a0-7498-4db1-b32e-613df6c3f987/a5acd85e-3114-4004-a4be-0df8305cfbf6"
-      (reference "U?") (unit 1) (value "MAX485E") (footprint "")
-    )
     (path "/6fbcc029-2e97-4cbb-aefe-dadd6dac0b49/c24eb077-6d4a-4ccd-bd1c-9ae5a44d9429"
-      (reference "U?") (unit 1) (value "519") (footprint "")
-    )
-  )
+      (reference "U7") (unit 1) (value "519") (footprint "")
+    )
+    (path "/6fbcc029-2e97-4cbb-aefe-dadd6dac0b49/801548aa-1a6b-4b2f-a875-e509e4453ddf"
+      (reference "U8") (unit 1) (value "MAX485E") (footprint "")
+    )
+  )
