File: EECD-22-7/ultrasound_sch.kicad_sch (KiCad schematic)
At the start: 6 parts

Commit message: Add files via upload
Connections:
- net +1V0 renamed acoustic
Changed lines of the file:
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@@
     (stroke (width 0) (type default) (color 0 0 0 0))
+  )
+  (global_label "acoustic" (shape input) (at 64.77 81.28 180) (fields_autoplaced)
+    (effects (font (size 1.27 1.27)) (justify right))
+    (property "Intersheet References" "${INTERSHEET_REFS}" (id 0) (at 54.374 81.2006 0)
+      (effects (font (size 1.27 1.27)) (justify right) hide)
+    )
   )
   (symbol (lib_id "Device:R") (at 111.76 81.28 90) (unit 1)
@@
     (pin "2")
   )
-  (symbol (lib_id "power:+1V0") (at 64.77 81.28 270) (unit 1)
-    (in_bom yes) (on_board yes) (fields_autoplaced)
-    (property "Reference" "#PWR?" (id 0) (at 60.96 81.28 0)
-      (effects (font (size 1.27 1.27)) hide)
-    )
-    (property "Value" "+1V0" (id 1) (at 68.58 81.2799 90)
-      (effects (font (size 1.27 1.27)) (justify left))
-    )
-    (property "Footprint" "" (id 2) (at 64.77 81.28 0)
-      (effects (font (size 1.27 1.27)) hide)
-    )
-    (property "Datasheet" "" (id 3) (at 64.77 81.28 0)
-      (effects (font (size 1.27 1.27)) hide)
-    )
-    (pin "1")
-  )
   (symbol (lib_id "Device:C") (at 82.55 81.28 90) (unit 1)
