File: EECD-22-7/ultrasound_sch.kicad_sch (KiCad schematic)
At the start: 6 parts

Commit message: Add files via upload
Parts:
- renumbered C1 to C5, R1 to R2, R2 to R3
Changed lines of the file:
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@@
   (symbol (lib_id "Device:R") (at 111.76 81.28 90) (unit 1)
     (in_bom yes) (on_board yes) (fields_autoplaced)
-    (property "Reference" "R1" (id 0) (at 111.76 74.93 90))
+    (property "Reference" "R2" (id 0) (at 111.76 74.93 90))
     (property "Value" "100R" (id 1) (at 111.76 77.47 90))
     (property "Footprint" "" (id 2) (at 111.76 83.058 90)
@@
   (symbol (lib_id "Device:C") (at 82.55 81.28 90) (unit 1)
     (in_bom yes) (on_board yes) (fields_autoplaced)
-    (property "Reference" "C1" (id 0) (at 82.55 73.66 90))
+    (property "Reference" "C5" (id 0) (at 82.55 73.66 90))
     (property "Value" "0.1uF" (id 1) (at 82.55 76.2 90))
     (property "Footprint" "" (id 2) (at 86.36 80.3148 0)
@@
   (symbol (lib_id "Device:R") (at 119.38 91.44 0) (unit 1)
     (in_bom yes) (on_board yes) (fields_autoplaced)
-    (property "Reference" "R2" (id 0) (at 121.92 90.1699 0)
+    (property "Reference" "R3" (id 0) (at 121.92 90.1699 0)
       (effects (font (size 1.27 1.27)) (justify left))
     )
@@
   (symbol (lib_id "power:GND") (at 76.2 101.6 0) (unit 1)
     (in_bom yes) (on_board yes) (fields_autoplaced)
-    (property "Reference" "#PWR0102" (id 0) (at 76.2 107.95 0)
+    (property "Reference" "#PWR03" (id 0) (at 76.2 107.95 0)
       (effects (font (size 1.27 1.27)) hide)
     )

Commit message: Add files via upload
Parts:
- added J5: Screw_Terminal_01x02, TerminalBlock_MetzConnect:TerminalBlock_MetzConnect_Type055_RT01502HDWU_1x02_P5.00mm_Horizontal, symbol Connector:Screw_Terminal_01x02
- C5: footprint (none) -> Capacitor_SMD:C_0603_1608Metric
- R2, R3: footprint (none) -> Resistor_SMD:R_0603_1608Metric
Connections:
- net GND: now also J5.2 (Pin_2)
- net at BZ1.1 (-), R2.2, R3.1: now also J5.1 (Pin_1)
Changed lines of the file:
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@@
   (junction (at 90.17 81.28) (diameter 0) (color 0 0 0 0)
+  )
+  (junction (at 129.54 81.28) (diameter 0) (color 0 0 0 0)
   )
   (junction (at 90.17 101.6) (diameter 0) (color 0 0 0 0)
@@
   )
   (junction (at 119.38 101.6) (diameter 0) (color 0 0 0 0)
+  )
+  (junction (at 129.54 101.6) (diameter 0) (color 0 0 0 0)
   )
   (wire (pts (xy 104.14 96.52) (xy 104.14 101.6))
@@
     (stroke (width 0) (type default) (color 0 0 0 0))
   )
+  (wire (pts (xy 147.32 81.28) (xy 129.54 81.28))
+    (stroke (width 0) (type default) (color 0 0 0 0))
+  )
+  (wire (pts (xy 147.32 91.44) (xy 147.32 101.6))
+    (stroke (width 0) (type default) (color 0 0 0 0))
+  )
   (wire (pts (xy 90.17 101.6) (xy 76.2 101.6))
+    (stroke (width 0) (type default) (color 0 0 0 0))
+  )
+  (wire (pts (xy 147.32 88.9) (xy 147.32 81.28))
     (stroke (width 0) (type default) (color 0 0 0 0))
   )
@@
   )
   (wire (pts (xy 119.38 81.28) (xy 115.57 81.28))
+    (stroke (width 0) (type default) (color 0 0 0 0))
+  )
+  (wire (pts (xy 147.32 101.6) (xy 129.54 101.6))
     (stroke (width 0) (type default) (color 0 0 0 0))
   )
@@
     (property "Reference" "R2" (id 0) (at 111.76 74.93 90))
     (property "Value" "100R" (id 1) (at 111.76 77.47 90))
-    (property "Footprint" "" (id 2) (at 111.76 83.058 90)
+    (property "Footprint" "Resistor_SMD:R_0603_1608Metric" (id 2) (at 111.76 83.058 90)
       (effects (font (size 1.27 1.27)) hide)
     )
@@
     (property "Reference" "C5" (id 0) (at 82.55 73.66 90))
     (property "Value" "0.1uF" (id 1) (at 82.55 76.2 90))
-    (property "Footprint" "" (id 2) (at 86.36 80.3148 0)
+    (property "Footprint" "Capacitor_SMD:C_0603_1608Metric" (id 2) (at 86.36 80.3148 0)
       (effects (font (size 1.27 1.27)) hide)
     )
@@
     (pin "2")
   )
+  (symbol (lib_id "Connector:Screw_Terminal_01x02") (at 152.4 88.9 0) (unit 1)
+    (in_bom yes) (on_board yes) (fields_autoplaced)
+    (property "Reference" "J5" (id 0) (at 154.94 88.8999 0)
+      (effects (font (size 1.27 1.27)) (justify left))
+    )
+    (property "Value" "Screw_Terminal_01x02" (id 1) (at 154.94 91.4399 0)
+      (effects (font (size 1.27 1.27)) (justify left))
+    )
+    (property "Footprint" "TerminalBlock_MetzConnect:TerminalBlock_MetzConnect_Type055_RT01502HDWU_1x02_P5.00mm_Horizontal" (id 2) (at 152.4 88.9 0)
+      (effects (font (size 1.27 1.27)) hide)
+    )
+    (property "Datasheet" "~" (id 3) (at 152.4 88.9 0)
+      (effects (font (size 1.27 1.27)) hide)
+    )
+    (pin "1")
+    (pin "2")
+  )
   (symbol (lib_id "Device:Buzzer") (at 132.08 90.17 0) (unit 1)
-    (in_bom yes) (on_board yes) (fields_autoplaced)
+    (in_bom yes) (on_board no) (fields_autoplaced)
     (property "Reference" "BZ1" (id 0) (at 135.89 88.8999 0)
       (effects (font (size 1.27 1.27)) (justify left))
@@
       (effects (font (size 1.27 1.27)) (justify left))
     )
-    (property "Footprint" "" (id 2) (at 117.602 91.44 90)
+    (property "Footprint" "Resistor_SMD:R_0603_1608Metric" (id 2) (at 117.602 91.44 90)
       (effects (font (size 1.27 1.27)) hide)
     )
