File: EECD-22-7/mcu_sch.kicad_sch (KiCad schematic)
At the start: 1 part

Commit message: Add files via upload
Parts:
- removed U?: ATmega644V-10M, Package_DFN_QFN:QFN-44-1EP_7x7mm_P0.5mm_EP5.2x5.2mm, symbol MCU_Microchip_ATmega:ATmega644V-10M
- added U1: STM32F103CBUx, Package_DFN_QFN:QFN-48-1EP_7x7mm_P0.5mm_EP5.6x5.6mm, symbol MCU_ST_STM32F1:STM32F103CBUx
Changed lines of the file:
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@@
 (kicad_sch (version 20211123) (generator eeschema)
   (paper "A4")
-  (symbol (lib_id "MCU_Microchip_ATmega:ATmega644V-10M") (at 120.65 91.44 0) (unit 1)
+  (symbol (lib_id "MCU_ST_STM32F1:STM32F103CBUx") (at 152.4 82.55 0) (unit 1)
     (in_bom yes) (on_board yes) (fields_autoplaced)
-    (property "Reference" "U?" (id 0) (at 122.6694 142.24 0)
+    (property "Reference" "U1" (id 0) (at 159.4994 41.91 0)
       (effects (font (size 1.27 1.27)) (justify left))
     )
-    (property "Value" "ATmega644V-10M" (id 1) (at 122.6694 144.78 0)
+    (property "Value" "STM32F103CBUx" (id 1) (at 159.4994 44.45 0)
       (effects (font (size 1.27 1.27)) (justify left))
     )
-    (property "Footprint" "Package_DFN_QFN:QFN-44-1EP_7x7mm_P0.5mm_EP5.2x5.2mm" (id 2) (at 120.65 91.44 0)
-      (effects (font (size 1.27 1.27) italic) hide)
+    (property "Footprint" "Package_DFN_QFN:QFN-48-1EP_7x7mm_P0.5mm_EP5.6x5.6mm" (id 2) (at 137.16 118.11 0)
+      (effects (font (size 1.27 1.27)) (justify right) hide)
     )
-    (property "Datasheet" "http://ww1.microchip.com/downloads/en/DeviceDoc/doc2593.pdf" (id 3) (at 120.65 91.44 0)
+    (property "Datasheet" "http://www.st.com/st-web-ui/static/active/en/resource/technical/document/datasheet/CD00161566.pdf" (id 3) (at 152.4 82.55 0)
       (effects (font (size 1.27 1.27)) hide)
     )
@@
     (pin "44")
     (pin "45")
+    (pin "46")
+    (pin "47")
+    (pin "48")
+    (pin "49")
     (pin "5")
     (pin "6")

Commit message: Add files via upload
Parts:
- added C15, C16, C17, C19: 100nF, symbol pspice:C
- added C18: 10uF, symbol pspice:C
- added C20: 1uF, symbol pspice:C
- added R15: 10kR, symbol Device:R
- added R16: 500kR, symbol Device:R
- added SW1: SW_Push, symbol Switch:SW_Push
Connections:
- net 3.3V_out: now reaches U1.23 (VSS)
- net 3.3V_out: now also U1.35 (VSS), U1.47 (VSS), U1.49 (VSS), U1.8 (VSSA), C15.2, C16.2, C17.2, C18.2, C19.2, C20.2, R16.2
- net +3.3V: now reaches U1.24 (VDD)
- net +3.3V: now also U1.36 (VDD), U1.48 (VDD), U1.9 (VDDA), C15.1, C16.1, C17.1, C18.1, C19.1, C20.1, SW1.1
- net at U1.44 (BOOT0): now also R15.1
- new net: R15.2, R16.1, SW1.2

Commit message: Add files via upload
Connections:
- net +3.3V: now also U1.1 (VBAT)
- net 3.3V_out: no longer C15.2, C16.2, C17.2, C18.2, C19.2, C20.2, U1.23 (VSS), U1.35 (VSS), U1.47 (VSS), U1.49 (VSS), U1.8 (VSSA)
- new net 3.3V_GND: C15.2, C16.2, C17.2, C18.2, U1.23 (VSS), U1.35 (VSS), U1.47 (VSS), U1.49 (VSS)
- new net GND3.3V: C19.2, C20.2, U1.8 (VSSA)
Changed lines of the file:
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@@
   (junction (at 60.96 101.6) (diameter 0) (color 0 0 0 0)
+  )
+  (junction (at 147.32 39.37) (diameter 0) (color 0 0 0 0)
   )
   (junction (at 60.96 55.88) (diameter 0) (color 0 0 0 0)
@@
   )
   (wire (pts (xy 78.74 101.6) (xy 60.96 101.6))
+    (stroke (width 0) (type default) (color 0 0 0 0))
+  )
+  (wire (pts (xy 147.32 39.37) (xy 149.86 39.37))
     (stroke (width 0) (type default) (color 0 0 0 0))
   )
@@
     (stroke (width 0) (type default) (color 0 0 0 0))
   )
-  (wire (pts (xy 78.74 39.37) (xy 149.86 39.37))
+  (wire (pts (xy 78.74 39.37) (xy 147.32 39.37))
+    (stroke (width 0) (type default) (color 0 0 0 0))
+  )
+  (wire (pts (xy 147.32 39.37) (xy 147.32 44.45))
     (stroke (width 0) (type default) (color 0 0 0 0))
   )
@@
     )
   )
-  (global_label "3.3V_out" (shape input) (at 29.21 101.6 180) (fields_autoplaced)
+  (global_label "3.3V_GND" (shape input) (at 29.21 101.6 180) (fields_autoplaced)
     (effects (font (size 1.27 1.27)) (justify right))
-    (property "Intersheet References" "${INTERSHEET_REFS}" (id 0) (at 18.6931 101.5206 0)
+    (property "Intersheet References" "${INTERSHEET_REFS}" (id 0) (at 17.8464 101.5206 0)
       (effects (font (size 1.27 1.27)) (justify right) hide)
     )
@@
     )
   )
-  (global_label "3.3V_out" (shape input) (at 252.73 91.44 0) (fields_autoplaced)
+  (global_label "GND3.3V" (shape input) (at 252.73 91.44 0) (fields_autoplaced)
     (effects (font (size 1.27 1.27)) (justify left))
-    (property "Intersheet References" "${INTERSHEET_REFS}" (id 0) (at 263.2469 91.3606 0)
+    (property "Intersheet References" "${INTERSHEET_REFS}" (id 0) (at 263.126 91.3606 0)
       (effects (font (size 1.27 1.27)) (justify left) hide)
     )

Commit message: Add files via upload
Connections:
- net 3.3V_GND is gone; now on net 3.3V_out: C15.2, C16.2, C17.2, C18.2, U1.23 (VSS), U1.35 (VSS), U1.47 (VSS), U1.49 (VSS)
- net GND3.3V is gone; now on net 3.3V_out: C19.2, C20.2, U1.8 (VSSA)
- net +3.3V: no longer U1.1 (VBAT)
- net SPI_SCLK: now reaches U1.15 (PA5)
- net SPI_SDI: now reaches U1.16 (PA6)
- net SPI_SDO: now reaches U1.17 (PA7)
- net GPIO_1: now reaches U1.18 (PB0)
- net GPIO_2: now reaches U1.19 (PB1)
- net GPIO_3: now reaches U1.20 (PB2)
- net GPIO_4: now reaches U1.39 (PB3)
- net GPIO_5: now reaches U1.40 (PB4)
- net I2C_1_CLK: now reaches U1.42 (PB6)
- net I2C_1_SDA: now reaches U1.43 (PB7)

Commit message: Add files via upload
Connections:
- net +3.3V: now also U1.1 (VBAT)
- net 3.3V_out: no longer C15.2, C16.2, C17.2, C18.2, C19.2, C20.2, U1.23 (VSS), U1.35 (VSS), U1.47 (VSS), U1.49 (VSS), U1.8 (VSSA)
- net GPIO_1 renamed temper
- net GPIO_2 renamed pres
- net GPIO_3 renamed acoustic
- net GPIO_4 renamed ch4_A
- net GPIO_5 renamed ch4_B
- net SPI_SCLK: no longer names the net of U1.15 (PA5)
- net SPI_SDI: no longer names the net of U1.16 (PA6)
- net SPI_SDO: no longer names the net of U1.17 (PA7)
- new net 3.3V_GND: C15.2, C16.2, C17.2, C18.2, U1.23 (VSS), U1.35 (VSS), U1.47 (VSS), U1.49 (VSS)
- new net GND3.3V: C19.2, C20.2, U1.8 (VSSA)

Commit message: Add files via upload
Parts:
- added C21: 100nF, symbol Device:C
Connections:
- net 3.3V_out is gone; now on net GND3.3V: R16.2
- net GND3.3V: now also C21.1
- net peri_power_1: now reaches U1.41 (PB5)
- net at R15.1, U1.44 (BOOT0): now also C21.2
- net peri_power_2: now reaches U1.45 (PB8)
- no-connect marks 0 -> 29
Other:
- moved on the sheet: R15, R16, SW1

Commit message: Add files via upload
Parts:
- added J3: Conn_ARM_JTAG_SWD_10, Connector_PinHeader_1.27mm:PinHeader_2x05_P1.27mm_Horizontal, symbol Connector:Conn_ARM_JTAG_SWD_10
Connections:
- net +3.3V: now also J3.1 (VTref)
- net GND3.3V: now also J3.3 (GND), J3.5 (GND)
- net ch4_A: now also U1.46 (PB9); no longer U1.39 (PB3)
- net SWDIO: now reaches U1.34 (PA13)
- net SWDIO: now also J3.2 (SWDIO/TMS)
- net SWDLK: now reaches U1.37 (PA14)
- net SWDLK: now also J3.4 (SWDCLK/TCK)
- net TDI: now reaches U1.38 (PA15)
- net TDI: now also J3.8 (NC/TDI)
- net RST: now reaches U1.7 (NRST)
- net RST: now also J3.10 (~{RESET})
- new net TDO: J3.6 (SWO/TDO), U1.39 (PB3)
- no-connect marks 29 -> 25
