File: EECD-22-7/mcu_sch.kicad_sch (KiCad schematic)
At the start: 12 parts, among them J4 Conn_ARM_JTAG_SWD_10, SW1 SW_Push, U10 STM32F103CBUx

Commit message: Add files via upload
Parts:
- C18, C19, C20, C21, C22, C23, C24: footprint (none) -> Capacitor_SMD:C_0603_1608Metric
- R12, R13: footprint (none) -> Resistor_SMD:R_0603_1608Metric
- SW1: footprint (none) -> Button_Switch_SMD:SW_Push_1P1T_NO_6x6mm_H9.5mm
Changed lines of the file:
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@@
       (effects (font (size 1.27 1.27)) (justify left))
     )
-    (property "Footprint" "" (id 2) (at 78.74 78.74 0)
+    (property "Footprint" "Capacitor_SMD:C_0603_1608Metric" (id 2) (at 78.74 78.74 0)
       (effects (font (size 1.27 1.27)) hide)
     )
@@
       (effects (font (size 1.27 1.27)) (justify left))
     )
-    (property "Footprint" "" (id 2) (at 108.712 60.96 90)
+    (property "Footprint" "Resistor_SMD:R_0603_1608Metric" (id 2) (at 108.712 60.96 90)
       (effects (font (size 1.27 1.27)) hide)
     )
@@
     (property "Reference" "SW1" (id 0) (at 102.87 46.99 0))
     (property "Value" "SW_Push" (id 1) (at 102.87 49.53 0))
-    (property "Footprint" "" (id 2) (at 102.87 49.53 0)
+    (property "Footprint" "Button_Switch_SMD:SW_Push_1P1T_NO_6x6mm_H9.5mm" (id 2) (at 102.87 49.53 0)
       (effects (font (size 1.27 1.27)) hide)
     )
@@
       (effects (font (size 1.27 1.27)) (justify right))
     )
-    (property "Footprint" "" (id 2) (at 130.5052 54.61 0)
+    (property "Footprint" "Capacitor_SMD:C_0603_1608Metric" (id 2) (at 130.5052 54.61 0)
       (effects (font (size 1.27 1.27)) hide)
     )
@@
       (effects (font (size 1.27 1.27)) (justify left))
     )
-    (property "Footprint" "" (id 2) (at 252.73 78.74 0)
+    (property "Footprint" "Capacitor_SMD:C_0603_1608Metric" (id 2) (at 252.73 78.74 0)
       (effects (font (size 1.27 1.27)) hide)
     )
@@
       (effects (font (size 1.27 1.27)) (justify left))
     )
-    (property "Footprint" "" (id 2) (at 232.41 78.74 0)
+    (property "Footprint" "Capacitor_SMD:C_0603_1608Metric" (id 2) (at 232.41 78.74 0)
       (effects (font (size 1.27 1.27)) hide)
     )
@@
       (effects (font (size 1.27 1.27)) (justify left))
     )
-    (property "Footprint" "" (id 2) (at 60.96 78.74 0)
+    (property "Footprint" "Capacitor_SMD:C_0603_1608Metric" (id 2) (at 60.96 78.74 0)
       (effects (font (size 1.27 1.27)) hide)
     )
@@
     (property "Reference" "R12" (id 0) (at 116.84 48.26 90))
     (property "Value" "10kR" (id 1) (at 116.84 50.8 90))
-    (property "Footprint" "" (id 2) (at 116.84 52.832 90)
+    (property "Footprint" "Resistor_SMD:R_0603_1608Metric" (id 2) (at 116.84 52.832 90)
       (effects (font (size 1.27 1.27)) hide)
     )
@@
       (effects (font (size 1.27 1.27)) (justify left))
     )
-    (property "Footprint" "" (id 2) (at 29.21 78.74 0)
+    (property "Footprint" "Capacitor_SMD:C_0603_1608Metric" (id 2) (at 29.21 78.74 0)
       (effects (font (size 1.27 1.27)) hide)
     )
@@
       (effects (font (size 1.27 1.27)) (justify left))
     )
-    (property "Footprint" "" (id 2) (at 45.72 78.74 0)
+    (property "Footprint" "Capacitor_SMD:C_0603_1608Metric" (id 2) (at 45.72 78.74 0)
       (effects (font (size 1.27 1.27)) hide)
     )
