File: EECD-22-7/measurements_sch.kicad_sch (KiCad schematic)
At the start: 5 parts, among them J1_I2C_Gamma_Sensor? Conn_01x06_Female, U1_Pressure_Sensor? MS5525DSO, U2_Temperature_Sensor? TMP1075D, U7 519, U8 MAX485E

Commit message: Add files via upload
Parts:
- removed U1_Pressure_Sensor?: MS5525DSO, symbol Sensor_Pressure:MS5525DSO
- removed U2_Temperature_Sensor?: TMP1075D, Package_SO:SO-8_3.9x4.9mm_P1.27mm, symbol Sensor_Temperature:TMP1075D
- added C25: 100nF, symbol Device:C
- added R25: 4.7KR, symbol Device:R
- added U8: DS18B20, Package_TO_SOT_THT:TO-92_Inline, symbol Sensor_Temperature:DS18B20
Connections:
- new net +5v: C25.1, R25.1, U8.3 (VDD)
- new net GND5V: C25.2, U8.1 (GND)
- new net temper: R25.2, U8.2 (DQ)
Changed lines of the file:
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@@
 (kicad_sch (version 20211123) (generator eeschema)
   (paper "A4")
+  (junction (at 190.5 96.52) (diameter 0) (color 0 0 0 0)
+  )
+  (junction (at 218.44 81.28) (diameter 0) (color 0 0 0 0)
+  )
+  (junction (at 228.6 88.9) (diameter 0) (color 0 0 0 0)
+  )
+  (junction (at 190.5 81.28) (diameter 0) (color 0 0 0 0)
+  )
+  (wire (pts (xy 190.5 92.71) (xy 190.5 96.52))
+    (stroke (width 0) (type default) (color 0 0 0 0))
+  )
+  (wire (pts (xy 226.06 88.9) (xy 228.6 88.9))
+    (stroke (width 0) (type default) (color 0 0 0 0))
+  )
+  (wire (pts (xy 190.5 81.28) (xy 218.44 81.28))
+    (stroke (width 0) (type default) (color 0 0 0 0))
+  )
+  (wire (pts (xy 187.96 81.28) (xy 190.5 81.28))
+    (stroke (width 0) (type default) (color 0 0 0 0))
+  )
+  (wire (pts (xy 228.6 88.9) (xy 238.76 88.9))
+    (stroke (width 0) (type default) (color 0 0 0 0))
+  )
+  (wire (pts (xy 190.5 81.28) (xy 190.5 85.09))
+    (stroke (width 0) (type default) (color 0 0 0 0))
+  )
+  (wire (pts (xy 190.5 96.52) (xy 218.44 96.52))
+    (stroke (width 0) (type default) (color 0 0 0 0))
+  )
+  (wire (pts (xy 189.23 96.52) (xy 190.5 96.52))
+    (stroke (width 0) (type default) (color 0 0 0 0))
+  )
+  (wire (pts (xy 218.44 81.28) (xy 228.6 81.28))
+    (stroke (width 0) (type default) (color 0 0 0 0))
+  )
+  (global_label "temper" (shape input) (at 238.76 88.9 0) (fields_autoplaced)
+    (effects (font (size 1.27 1.27)) (justify left))
+    (property "Intersheet References" "${INTERSHEET_REFS}" (id 0) (at 247.7045 88.8206 0)
+      (effects (font (size 1.27 1.27)) (justify left) hide)
+    )
+  )
+  (global_label "GND5V" (shape input) (at 189.23 96.52 180) (fields_autoplaced)
+    (effects (font (size 1.27 1.27)) (justify right))
+    (property "Intersheet References" "${INTERSHEET_REFS}" (id 0) (at 180.6483 96.4406 0)
+      (effects (font (size 1.27 1.27)) (justify right) hide)
+    )
+  )
+  (global_label "+5v" (shape input) (at 187.96 81.28 180) (fields_autoplaced)
+    (effects (font (size 1.27 1.27)) (justify right))
+    (property "Intersheet References" "${INTERSHEET_REFS}" (id 0) (at 181.7974 81.2006 0)
+      (effects (font (size 1.27 1.27)) (justify right) hide)
+    )
+  )
   (symbol (lib_id "Connector:Conn_01x06_Female") (at 140.97 132.08 0) (unit 1)
     (in_bom yes) (on_board yes) (fields_autoplaced)
@@
     (pin "6")
   )
-  (symbol (lib_id "Sensor_Temperature:TMP1075D") (at 236.982 125.984 0) (unit 1)
+  (symbol (lib_id "Device:R") (at 228.6 85.09 0) (unit 1)
     (in_bom yes) (on_board yes) (fields_autoplaced)
-    (property "Reference" "U2_Temperature_Sensor?" (id 0) (at 239.0014 115.824 0)
+    (property "Reference" "R25" (id 0) (at 231.14 83.8199 0)
       (effects (font (size 1.27 1.27)) (justify left))
     )
-    (property "Value" "TMP1075D" (id 1) (at 239.0014 118.364 0)
+    (property "Value" "4.7KR" (id 1) (at 231.14 86.3599 0)
       (effects (font (size 1.27 1.27)) (justify left))
     )
-    (property "Footprint" "Package_SO:SO-8_3.9x4.9mm_P1.27mm" (id 2) (at 236.982 132.334 0)
+    (property "Footprint" "" (id 2) (at 226.822 85.09 90)
       (effects (font (size 1.27 1.27)) hide)
     )
-    (property "Datasheet" "https://www.ti.com/lit/gpn/tmp1075" (id 3) (at 236.982 125.984 0)
+    (property "Datasheet" "~" (id 3) (at 228.6 85.09 0)
+      (effects (font (size 1.27 1.27)) hide)
+    )
+    (pin "1")
+    (pin "2")
+  )
+  (symbol (lib_id "Sensor_Temperature:DS18B20") (at 218.44 88.9 0) (unit 1)
+    (in_bom yes) (on_board yes) (fields_autoplaced)
+    (property "Reference" "U8" (id 0) (at 212.09 87.6299 0)
+      (effects (font (size 1.27 1.27)) (justify right))
+    )
+    (property "Value" "DS18B20" (id 1) (at 212.09 90.1699 0)
+      (effects (font (size 1.27 1.27)) (justify right))
+    )
+    (property "Footprint" "Package_TO_SOT_THT:TO-92_Inline" (id 2) (at 193.04 95.25 0)
+      (effects (font (size 1.27 1.27)) hide)
+    )
+    (property "Datasheet" "http://datasheets.maximintegrated.com/en/ds/DS18B20.pdf" (id 3) (at 214.63 82.55 0)
       (effects (font (size 1.27 1.27)) hide)
     )
@@
     (pin "2")
     (pin "3")
-    (pin "4")
-    (pin "5")
-    (pin "6")
-    (pin "7")
-    (pin "8")
   )
   (symbol (lib_id "Interface_UART:MAX485E") (at 140.97 88.9 0) (unit 1)
@@
     (pin "8")
   )
-  (symbol (lib_id "Sensor_Pressure:MS5525DSO") (at 241.554 91.44 0) (unit 1)
-    (in_bom yes) (on_board yes) (fields_autoplaced)
-    (property "Reference" "U1_Pressure_Sensor?" (id 0) (at 243.5734 76.2 0)
-      (effects (font (size 1.27 1.27)) (justify left))
-    )
-    (property "Value" "MS5525DSO" (id 1) (at 243.5734 78.74 0)
-      (effects (font (size 1.27 1.27)) (justify left))
-    )
-    (property "Footprint" "" (id 2) (at 241.554 105.41 0)
-      (effects (font (size 1.27 1.27)) hide)
-    )
-    (property "Datasheet" "https://www.te.com/commerce/DocumentDelivery/DDEController?Action=srchrtrv&DocNm=MS5525DSO&DocType=DS&DocLang=English" (id 3) (at 241.554 107.95 0)
-      (effects (font (size 1.27 1.27)) hide)
-    )
-    (pin "1")
-    (pin "10")
-    (pin "11")
-    (pin "12")
-    (pin "13")
-    (pin "14")
-    (pin "2")
-    (pin "3")
-    (pin "4")
-    (pin "5")
-    (pin "6")
-    (pin "7")
-    (pin "8")
-    (pin "9")
-  )
   (symbol (lib_id "Analog:519") (at 50.8 91.44 0) (unit 1)
     (in_bom yes) (on_board no) (fields_autoplaced)
@@
     (pin "4")
   )
+  (symbol (lib_id "Device:C") (at 190.5 88.9 0) (unit 1)
+    (in_bom yes) (on_board yes) (fields_autoplaced)
+    (property "Reference" "C25" (id 0) (at 194.31 87.6299 0)
+      (effects (font (size 1.27 1.27)) (justify left))
+    )
+    (property "Value" "100nF" (id 1) (at 194.31 90.1699 0)
+      (effects (font (size 1.27 1.27)) (justify left))
+    )
+    (property "Footprint" "" (id 2) (at 191.4652 92.71 0)
+      (effects (font (size 1.27 1.27)) hide)
+    )
+    (property "Datasheet" "~" (id 3) (at 190.5 88.9 0)
+      (effects (font (size 1.27 1.27)) hide)
+    )
+    (pin "1")
+    (pin "2")
+  )
 )

Commit message: Add files via upload
Parts:
- added C26, C27: 100nF, symbol Device:C
- added U10: 4002B, symbol Comparator:4002B
- added U9: Mets_methane_sensor, symbol methane:Mets_methane_sensor
- U7: value 519 -> 519.933.003M
Connections:
- net at U8.1 (RO): now also U9. (RO)
- net at U8.2 (~{RE}): now also U9. (RO)
- net at U8.3 (DE): now also U9. (RO)
- net at U8.4 (DI): now also U9. (RO)
- net GND12V: now reaches U8.5 (GND)
- net GND12V: now also C26.2, C27.2, U10. (OUT_PCB,)
- net ch4_A: now reaches U8.6 (A)
- net ch4_B: now reaches U8.7 (B)
- net +12V: now reaches U8.8 (VCC)
- net +12V: now also C26.1, C27.1, U10. (OUT_PCB,)
- net at U7.1 (IN): now also U10.1 (IN_M12)
- net at U7.3 (GND): now also U10.3 (GND_M12)
- net at U7.4 (OUT): now also U10.4 (OUT_M12)
- new net pres: U10. (OUT_PCB,)
Other:
- moved on the sheet: C25, J1_I2C_Gamma_Sensor?, R25, U7, U8

Commit message: Add files via upload
Parts:
- removed C25, C26, C27: 100nF, symbol Device:C
- removed R25: 4.7KR, symbol Device:R
- removed U10: 4002B, symbol Comparator:4002B
- removed U8: DS18B20, Package_TO_SOT_THT:TO-92_Inline, symbol Sensor_Temperature:DS18B20
- removed U9: Mets_methane_sensor, symbol methane:Mets_methane_sensor
- added C? (x5): 100nF, symbol Device:C
- added U1_Pressure_Sensor?: MS5525DSO, symbol Sensor_Pressure:MS5525DSO
- added U2_Temperature_Sensor?: TMP1075D, Package_SO:SO-8_3.9x4.9mm_P1.27mm, symbol Sensor_Temperature:TMP1075D
- U7: value 519.933.003M -> 519
Connections:
- net GND12V is gone; now on net Earth: U8.5 (GND)
- net 5V: now reaches J1_I2C_Gamma_Sensor?.3 (Pin_3)
- net 5V: now also C?.2, C?.2
- net Earth: now reaches J1_I2C_Gamma_Sensor?.4 (Pin_4)
- net Earth: now also U7.3 (GND), C?.1, C?.1, C?.1, C?.2
- net I2C_1_SDA: now reaches J1_I2C_Gamma_Sensor?.5 (Pin_5)
- net I2C_1_CLK: now reaches J1_I2C_Gamma_Sensor?.6 (Pin_6)
- net GPIO_4: now reaches U8.1 (RO)
- net GPIO_5: now reaches U8.2 (~{RE})
- net GPIO_6: now reaches U7.4 (OUT)
- net +12V: no longer names the net of U8.8 (VCC)
- net +12V: now also C?.1
- net ch4_A renamed GPIO_3
- net GPIO_3: now also U2_Temperature_Sensor?.3 (ALERT)
- net ch4_B: no longer names the net of U8.7 (B)
- new net: U1_Pressure_Sensor?.1 (SIN-), U1_Pressure_Sensor?.3 (SIN-)
- new net: U1_Pressure_Sensor?.8 (CSB), U1_Pressure_Sensor?.9 (SUPPLY-)
- new net 3.3V: C?.2, U1_Pressure_Sensor?.11 (SUPPLY+), U1_Pressure_Sensor?.13 (SUPPLY+), U2_Temperature_Sensor?.8 (V+)
- new net GND: C?.1, U2_Temperature_Sensor?.5 (A2), U2_Temperature_Sensor?.6 (A1), U2_Temperature_Sensor?.7 (A0)
- new net GPIO_1: U1_Pressure_Sensor?.12 (SOUT+), U1_Pressure_Sensor?.14 (SOUT+)
- new net GPIO_2: U1_Pressure_Sensor?.2 (SOUT-), U1_Pressure_Sensor?.4 (SOUT-)
- new net I2C_2_CLK: U2_Temperature_Sensor?.2 (SCL)
- new net I2C_2_SDA: U2_Temperature_Sensor?.1 (SDA)
- new net SPI_SCLK: U1_Pressure_Sensor?.7 (SCLK/SCL)
- new net SPI_SDI: U1_Pressure_Sensor?.6 (SDI/SDA)
- new net SPI_SDO: U1_Pressure_Sensor?.5 (SDO)
Other:
- moved on the sheet: J1_I2C_Gamma_Sensor?, U7, U8

Commit message: Add files via upload
Parts:
- removed C? (x5): 100nF, symbol Device:C
- removed J1_I2C_Gamma_Sensor?: Conn_01x06_Female, symbol Connector:Conn_01x06_Female
- removed U1_Pressure_Sensor?: MS5525DSO, symbol Sensor_Pressure:MS5525DSO
- removed U2_Temperature_Sensor?: TMP1075D, Package_SO:SO-8_3.9x4.9mm_P1.27mm, symbol Sensor_Temperature:TMP1075D
- added C25, C26, C27, C?: 100nF, symbol Device:C
- added J1_I2C_Gamma_Sensor?: Conn_01x06_Female, symbol Connector:Conn_01x06_Female
- added R25: 4.7KR, symbol Device:R
- added U10: 4002B, symbol Comparator:4002B
- added U8: DS18B20, Package_TO_SOT_THT:TO-92_Inline, symbol Sensor_Temperature:DS18B20
- added U9: Mets_methane_sensor, symbol methane:Mets_methane_sensor
- U7: value 519 -> 519.933.003M
Connections:
- net 5V: now also C?.2, J1_I2C_Gamma_Sensor?.3 (Pin_3)
- net Earth: now also C?.1, J1_I2C_Gamma_Sensor?.4 (Pin_4); no longer U7.3 (GND), U8.5 (GND)
- net I2C_1_CLK: now also J1_I2C_Gamma_Sensor?.6 (Pin_6)
- net I2C_1_SDA: now also J1_I2C_Gamma_Sensor?.5 (Pin_5)
- net at U8.3 (DE): now also U9. (RO)
- net at U8.4 (DI): now also U9. (RO)
- net ch4_B: now reaches U8.7 (B)
- net +12V: now reaches U8.8 (VCC)
- net +12V: now also C26.1, C27.1, U10. (OUT_PCB,)
- net at U7.1 (IN): now also U10.1 (IN_M12)
- net GPIO_3 renamed ch4_A
- net GPIO_4: no longer names the net of U8.1 (RO)
- net GPIO_4: now also U9. (RO)
- net GPIO_5: no longer names the net of U8.2 (~{RE})
- net GPIO_5: now also U9. (RO)
- net GPIO_6: no longer names the net of U7.4 (OUT)
- net GPIO_6: now also U10.4 (OUT_M12)
- new net: U10.3 (GND_M12), U7.3 (GND)
- new net +5v: C25.1, R25.1, U8.3 (VDD)
- new net GND12V: C26.2, C27.2, U10. (OUT_PCB,), U8.5 (GND)
- new net GND5V: C25.2, U8.1 (GND)
- new net pres: U10. (OUT_PCB,)
- new net temper: R25.2, U8.2 (DQ)
Other:
- moved on the sheet: U7, U8

Commit message: Add files via upload
Parts:
- removed C?: 100nF, symbol Device:C
- added C26: 100nF, symbol Device:C
- added J2: Screw_Terminal_01x03, TerminalBlock_MetzConnect:TerminalBlock_MetzConnect_Type055_RT01503HDWU_1x03_P5.00mm_Horizontal, symbol Connector:Screw_Terminal_01x03
- added J3: Screw_Terminal_01x04, TerminalBlock_MetzConnect:TerminalBlock_MetzConnect_Type055_RT01504HDWU_1x04_P5.00mm_Horizontal, symbol Connector:Screw_Terminal_01x04
- U12: renamed from J1_I2C_Gamma_Sensor?; value Conn_01x06_Female -> GDK101
- renumbered C26 to C30, U8 to U11
Connections:
- net 5V is gone; now on net +5V: U12.3 (VCC)
- net GND5V: now also J2.2 (Pin_2)
- net I2C_1_CLK: now also J3.4 (Pin_4)
- net I2C_1_SDA: now also J3.3 (Pin_3)
- net temper: now also J2.3 (Pin_3)
- net +5v renamed +5V
- net +5V: now also C26.1, J2.1 (Pin_1), J3.1 (Pin_1)
- net Earth renamed GND
- net GND: now also C26.2, J3.2 (Pin_2)
- no-connect marks 0 -> 2

Commit message: Add files via upload
Parts:
- renumbered C25 to C1, C30 to C2, C27 to C3, C26 to C4, J2 to J1, J3 to J2, R25 to R1, U10 to U1, U7 to U2, U8 to U3, U9 to U4, U11 to U5, U12 to U6
Changed lines of the file:
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@@
   (symbol (lib_id "power:GND") (at 233.68 142.24 0) (unit 1)
     (in_bom yes) (on_board yes) (fields_autoplaced)
-    (property "Reference" "#PWR0117" (id 0) (at 233.68 148.59 0)
+    (property "Reference" "#PWR02" (id 0) (at 233.68 148.59 0)
       (effects (font (size 1.27 1.27)) hide)
     )
@@
   (symbol (lib_id "Device:R") (at 231.14 68.58 0) (unit 1)
     (in_bom yes) (on_board yes) (fields_autoplaced)
-    (property "Reference" "R25" (id 0) (at 233.68 67.3099 0)
+    (property "Reference" "R1" (id 0) (at 233.68 67.3099 0)
       (effects (font (size 1.27 1.27)) (justify left))
     )
@@
   (symbol (lib_id "Device:C") (at 182.88 124.46 0) (unit 1)
     (in_bom yes) (on_board yes) (fields_autoplaced)
-    (property "Reference" "C26" (id 0) (at 186.69 123.1899 0)
+    (property "Reference" "C4" (id 0) (at 186.69 123.1899 0)
       (effects (font (size 1.27 1.27)) (justify left))
     )
@@
   )
   (symbol (lib_id "Sensor_Temperature:DS18B20") (at 220.98 72.39 0) (unit 1)
-    (in_bom yes) (on_board yes) (fields_autoplaced)
-    (property "Reference" "U8" (id 0) (at 214.63 71.1199 0)
+    (in_bom yes) (on_board no) (fields_autoplaced)
+    (property "Reference" "U3" (id 0) (at 214.63 71.1199 0)
       (effects (font (size 1.27 1.27)) (justify right))
     )
@@
   (symbol (lib_id "methane:Mets_methane_sensor") (at 52.07 113.03 0) (unit 1)
     (in_bom yes) (on_board yes) (fields_autoplaced)
-    (property "Reference" "U9" (id 0) (at 52.705 110.49 0))
+    (property "Reference" "U4" (id 0) (at 52.705 110.49 0))
     (property "Value" "Mets_methane_sensor" (id 1) (at 52.705 113.03 0))
     (property "Footprint" "" (id 2) (at 52.07 113.03 0)
@@
   (symbol (lib_id "power:GND") (at 204.47 128.27 0) (unit 1)
     (in_bom yes) (on_board yes) (fields_autoplaced)
-    (property "Reference" "#PWR0101" (id 0) (at 204.47 134.62 0)
+    (property "Reference" "#PWR01" (id 0) (at 204.47 134.62 0)
       (effects (font (size 1.27 1.27)) hide)
     )
@@
   (symbol (lib_id "Connector:Screw_Terminal_01x04") (at 251.46 142.24 0) (unit 1)
     (in_bom yes) (on_board yes) (fields_autoplaced)
-    (property "Reference" "J3" (id 0) (at 254 142.2399 0)
+    (property "Reference" "J2" (id 0) (at 254 142.2399 0)
       (effects (font (size 1.27 1.27)) (justify left))
     )
@@
   )
   (symbol (lib_id "Interface_UART:MAX485E") (at 74.93 119.38 0) (unit 1)
-    (in_bom yes) (on_board yes) (fields_autoplaced)
-    (property "Reference" "U11" (id 0) (at 76.9494 104.14 0)
+    (in_bom yes) (on_board no) (fields_autoplaced)
+    (property "Reference" "U5" (id 0) (at 76.9494 104.14 0)
       (effects (font (size 1.27 1.27)) (justify left))
     )
@@
   (symbol (lib_id "Connector:Screw_Terminal_01x03") (at 228.6 53.34 0) (unit 1)
     (in_bom yes) (on_board yes) (fields_autoplaced)
-    (property "Reference" "J2" (id 0) (at 231.14 52.0699 0)
+    (property "Reference" "J1" (id 0) (at 231.14 52.0699 0)
       (effects (font (size 1.27 1.27)) (justify left))
     )
@@
   (symbol (lib_id "Device:C") (at 101.6 119.38 0) (unit 1)
     (in_bom yes) (on_board yes) (fields_autoplaced)
-    (property "Reference" "C27" (id 0) (at 105.41 118.1099 0)
+    (property "Reference" "C3" (id 0) (at 105.41 118.1099 0)
       (effects (font (size 1.27 1.27)) (justify left))
     )
@@
   (symbol (lib_id "Device:C") (at 96.52 73.66 0) (unit 1)
     (in_bom yes) (on_board yes) (fields_autoplaced)
-    (property "Reference" "C30" (id 0) (at 100.33 72.3899 0)
+    (property "Reference" "C2" (id 0) (at 100.33 72.3899 0)
       (effects (font (size 1.27 1.27)) (justify left))
     )
@@
   (symbol (lib_id "Analog:519") (at 40.64 69.85 0) (unit 1)
     (in_bom yes) (on_board no)
-    (property "Reference" "U7" (id 0) (at 41.91 58.42 0))
+    (property "Reference" "U2" (id 0) (at 41.91 58.42 0))
     (property "Value" "519.933.003M" (id 1) (at 41.91 60.96 0))
     (property "Footprint" "" (id 2) (at 40.64 69.85 0)
@@
   (symbol (lib_id "Device:C") (at 193.04 72.39 0) (unit 1)
     (in_bom yes) (on_board yes) (fields_autoplaced)
-    (property "Reference" "C25" (id 0) (at 196.85 71.1199 0)
+    (property "Reference" "C1" (id 0) (at 196.85 71.1199 0)
       (effects (font (size 1.27 1.27)) (justify left))
     )
@@
   (symbol (lib_id "Connector:Conn_01x06_Female") (at 232.41 125.73 0) (unit 1)
     (in_bom yes) (on_board yes) (fields_autoplaced)
-    (property "Reference" "U12" (id 0) (at 231.14 115.57 0)
+    (property "Reference" "U6" (id 0) (at 231.14 115.57 0)
       (effects (font (size 1.27 1.27)) (justify left))
     )
@@
   (symbol (lib_name "4002B_1") (lib_id "Comparator:4002B") (at 78.74 59.69 0) (unit 1)
     (in_bom yes) (on_board yes) (fields_autoplaced)
-    (property "Reference" "U10" (id 0) (at 79.375 57.15 0))
+    (property "Reference" "U1" (id 0) (at 79.375 57.15 0))
     (property "Value" "4002B" (id 1) (at 79.375 59.69 0))
     (property "Footprint" "" (id 2) (at 78.74 59.69 0)
