File: EECD-22-7/measurements_sch.kicad_sch (KiCad schematic)
At the start: 13 parts, among them J1 Screw_Terminal_01x03, J2 Screw_Terminal_01x04, U1 4002B, U2 519.933.003M, U3 DS18B20, U4 Mets_methane_sensor, U5 MAX485E, U6 GDK101

Commit message: Add files via upload
Parts:
- C1, C2, C3, C4: footprint (none) -> Capacitor_SMD:C_0603_1608Metric
- R1: footprint (none) -> Resistor_SMD:R_0603_1608Metric
- U1: footprint (none) -> m12:m12con
Connections:
- net +12V: now also U1.5 (GND_PCB); no longer U1. (OUT_PCB,)
- net GND12V: now also U1.6 (IN_PCB); no longer U1. (OUT_PCB,)
- net pres: now also U1.2 (OUT_PCB,); no longer U1. (OUT_PCB,)
Changed lines of the file:
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@@
       (effects (font (size 1.27 1.27)) (justify left))
     )
-    (property "Footprint" "" (id 2) (at 229.362 68.58 90)
+    (property "Footprint" "Resistor_SMD:R_0603_1608Metric" (id 2) (at 229.362 68.58 90)
       (effects (font (size 1.27 1.27)) hide)
     )
@@
       (effects (font (size 1.27 1.27)) (justify left))
     )
-    (property "Footprint" "" (id 2) (at 183.8452 128.27 0)
+    (property "Footprint" "Capacitor_SMD:C_0603_1608Metric" (id 2) (at 183.8452 128.27 0)
       (effects (font (size 1.27 1.27)) hide)
     )
@@
   )
   (symbol (lib_id "methane:Mets_methane_sensor") (at 52.07 113.03 0) (unit 1)
-    (in_bom yes) (on_board yes) (fields_autoplaced)
+    (in_bom yes) (on_board no) (fields_autoplaced)
     (property "Reference" "U4" (id 0) (at 52.705 110.49 0))
     (property "Value" "Mets_methane_sensor" (id 1) (at 52.705 113.03 0))
@@
       (effects (font (size 1.27 1.27)) (justify left))
     )
-    (property "Footprint" "" (id 2) (at 102.5652 123.19 0)
+    (property "Footprint" "Capacitor_SMD:C_0603_1608Metric" (id 2) (at 102.5652 123.19 0)
       (effects (font (size 1.27 1.27)) hide)
     )
@@
       (effects (font (size 1.27 1.27)) (justify left))
     )
-    (property "Footprint" "" (id 2) (at 97.4852 77.47 0)
+    (property "Footprint" "Capacitor_SMD:C_0603_1608Metric" (id 2) (at 97.4852 77.47 0)
       (effects (font (size 1.27 1.27)) hide)
     )
@@
       (effects (font (size 1.27 1.27)) (justify left))
     )
-    (property "Footprint" "" (id 2) (at 194.0052 76.2 0)
+    (property "Footprint" "Capacitor_SMD:C_0603_1608Metric" (id 2) (at 194.0052 76.2 0)
       (effects (font (size 1.27 1.27)) hide)
     )
@@
   )
   (symbol (lib_id "Connector:Conn_01x06_Female") (at 232.41 125.73 0) (unit 1)
-    (in_bom yes) (on_board yes) (fields_autoplaced)
+    (in_bom yes) (on_board no) (fields_autoplaced)
     (property "Reference" "U6" (id 0) (at 231.14 115.57 0)
       (effects (font (size 1.27 1.27)) (justify left))
@@
       (effects (font (size 1.27 1.27)) (justify left))
     )
-    (property "Footprint" "" (id 2) (at 234.95 125.73 0))
+    (property "Footprint" "" (id 2) (at 234.95 125.73 0)
+      (effects (font (size 1.27 1.27)) hide)
+    )
     (property "Datasheet" "~" (id 3) (at 234.95 128.27 0)
       (effects (font (size 1.27 1.27)) hide)
@@
     (property "Reference" "U1" (id 0) (at 79.375 57.15 0))
     (property "Value" "4002B" (id 1) (at 79.375 59.69 0))
-    (property "Footprint" "" (id 2) (at 78.74 59.69 0)
+    (property "Footprint" "m12:m12con" (id 2) (at 78.74 59.69 0)
       (effects (font (size 1.27 1.27)) hide)
     )
@@
       (effects (font (size 1.27 1.27)) hide)
     )
-    (pin "")
-    (pin "")
-    (pin "")
-    (pin "1")
-    (pin "3")
-    (pin "4")
+    (pin "1")
+    (pin "2")
+    (pin "3")
+    (pin "4")
+    (pin "5")
+    (pin "6")
   )
   (sheet_instances
