File: EECD-22-7/_autosave-EECD-22-7.kicad_pcb (KiCad board)
At the start: 2 copper layers, 54 parts, among them J1 Screw_Terminal_01x03, J2 Screw_Terminal_01x04, J3 Screw_Terminal_01x02, J4 Conn_ARM_JTAG_SWD_10, Q1 IRF6616, Q2 IRF6616, SW1 SW_Push, U1 4002B, U10 STM32F103CBUx, U7 LMR54406DBVR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

Commit message: Add files via upload
Parts:
- added J5: Screw_Terminal_01x02, TerminalBlock_MetzConnect:TerminalBlock_MetzConnect_Type055_RT01502HDWU_1x02_P5.00mm_Horizontal, F.Cu at (149.9, 71.1)
Changed lines of the file:
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@@
+    )
+  )
+  (footprint "TerminalBlock_MetzConnect:TerminalBlock_MetzConnect_Type055_RT01502HDWU_1x02_P5.00mm_Horizontal" (layer "F.Cu")
+    (at 149.86 71.12)
+    (descr "terminal block Metz Connect Type055_RT01502HDWU, 2 pins, pitch 5mm, size 10x8mm^2, drill diamater 1.3mm, pad diameter 2.5mm, see http://www.metz-connect.com/de/system/files/productfiles/Datenblatt_310551_RT015xxHDWU_OFF-022723S.pdf, script-generated using https://github.com/pointhi/kicad-footprint-generator/scripts/TerminalBlock_MetzConnect")
+    (tags "THT terminal block Metz Connect Type055_RT01502HDWU pitch 5mm size 10x8mm^2 drill 1.3mm pad 2.5mm")
+    (property "Sheetfile" "ultrasound_sch.kicad_sch")
+    (property "Sheetname" "communication")
+    (attr through_hole)
+    (fp_text reference "J5" (at 2.5 -5.06) (layer "F.SilkS")
+      (effects (font (size 1 1) (thickness 0.15)))
+    )
+    (fp_text value "Screw_Terminal_01x02" (at 2.5 5.06) (layer "F.Fab")
+      (effects (font (size 1 1) (thickness 0.15)))
+    )
+    (fp_text user "${REFERENCE}" (at 2.5 3) (layer "F.Fab")
+      (effects (font (size 1 1) (thickness 0.15)))
+    )
+    (fp_line (start -2.56 -4.06) (end -2.56 4.06) (layer "F.SilkS") (width 0.12))
+    (fp_line (start -2.8 4.3) (end -0.8 4.3) (layer "F.SilkS") (width 0.12))
+    (fp_line (start -2.56 2) (end 7.56 2) (layer "F.SilkS") (width 0.12))
+    (fp_line (start 7.56 -4.06) (end 7.56 4.06) (layer "F.SilkS") (width 0.12))
+    (fp_line (start -2.56 -4.06) (end 7.56 -4.06) (layer "F.SilkS") (width 0.12))
+    (fp_line (start 6.07 -1.275) (end 6.011 -1.216) (layer "F.SilkS") (width 0.12))
+    (fp_line (start -2.56 -2) (end 7.56 -2) (layer "F.SilkS") (width 0.12))
+    (fp_line (start 6.275 -1.069) (end 6.181 -0.976) (layer "F.SilkS") (width 0.12))
+    (fp_line (start 3.99 1.216) (end 3.931 1.274) (layer "F.SilkS") (width 0.12))
+    (fp_line (start -2.8 2.06) (end -2.8 4.3) (layer "F.SilkS") (width 0.12))
+    (fp_line (start 3.82 0.976) (end 3.726 1.069) (layer "F.SilkS") (width 0.12))
+    (fp_line (start -2.56 4.06) (end 7.56 4.06) (layer "F.SilkS") (width 0.12))
+    (fp_arc (start 0.029383 1.68045) (mid -0.392304 1.634281) (end -0.789 1.484) (layer "F.SilkS") (width 0.12))
+    (fp_arc (start -1.483953 0.789089) (mid -1.680708 0.00005) (end -1.484 -0.789) (layer "F.SilkS") (width 0.12))
+    (fp_arc (start -0.789089 -1.483953) (mid -0.00005 -1.680708) (end 0.789 -1.484) (layer "F.SilkS") (width 0.12))
+    (fp_arc (start 0.788712 1.483352) (mid 0.406429 1.630097) (end 0 1.68) (layer "F.SilkS") (width 0.12))
+    (fp_arc (start 1.483953 -0.789089) (mid 1.680708 -0.00005) (end 1.484 0.789) (layer "F.SilkS") (width 0.12))
+    (fp_circle (center 5 0) (end 6.68 0) (layer "F.SilkS") (width 0.12) (fill none))
+    (fp_line (start -3 -4.5) (end -3 4.5) (layer "F.CrtYd") (width 0.05))
+    (fp_line (start 8 -4.5) (end -3 -4.5) (layer "F.CrtYd") (width 0.05))
+    (fp_line (start -3 4.5) (end 8 4.5) (layer "F.CrtYd") (width 0.05))
+    (fp_line (start 8 4.5) (end 8 -4.5) (layer "F.CrtYd") (width 0.05))
+    (fp_line (start -2.5 -2) (end 7.5 -2) (layer "F.Fab") (width 0.1))
+    (fp_line (start 7.5 4) (end -0.5 4) (layer "F.Fab") (width 0.1))
+    (fp_line (start -2.5 2) (end -2.5 -4) (layer "F.Fab") (width 0.1))
+    (fp_line (start 7.5 -4) (end 7.5 4) (layer "F.Fab") (width 0.1))
+    (fp_line (start -2.5 2) (end 7.5 2) (layer "F.Fab") (width 0.1))
+    (fp_line (start -0.5 4) (end -2.5 2) (layer "F.Fab") (width 0.1))
+    (fp_line (start 6.138 -0.955) (end 4.046 1.138) (layer "F.Fab") (width 0.1))
+    (fp_line (start -2.5 -4) (end 7.5 -4) (layer "F.Fab") (width 0.1))
+    (fp_line (start 1.138 -0.955) (end -0.955 1.138) (layer "F.Fab") (width 0.1))
+    (fp_line (start 5.955 -1.138) (end 3.863 0.955) (layer "F.Fab") (width 0.1))
+    (fp_line (start 0.955 -1.138) (end -1.138 0.955) (layer "F.Fab") (width 0.1))
+    (fp_circle (center 5 0) (end 6.5 0) (layer "F.Fab") (width 0.1) (fill none))
+    (fp_circle (center 0 0) (end 1.5 0) (layer "F.Fab") (width 0.1) (fill none))
+    (pad "1" thru_hole rect (at 0 0) (size 2.5 2.5) (drill 1.3) (layers *.Cu *.Mask)
+      (net 58 "Net-(BZ1-Pad1)") (pinfunction "Pin_1") (pintype "passive"))
+    (pad "2" thru_hole circle (at 5 0) (size 2.5 2.5) (drill 1.3) (layers *.Cu *.Mask)
+      (net 1 "GND12V") (pinfunction "Pin_2") (pintype "passive"))
+    (model "${KICAD6_3DMODEL_DIR}/TerminalBlock_MetzConnect.3dshapes/TerminalBlock_MetzConnect_Type055_RT01502HDWU_1x02_P5.00mm_Horizontal.wrl"
+      (offset (xyz 0 0 0))
+      (scale (xyz 1 1 1))
+      (rotate (xyz 0 0 0))
     )
   )
