File: EECD-22-7/EECD-22-7.kicad_pcb (KiCad board)
At the start: 2 copper layers, 54 parts, among them J1 Screw_Terminal_01x03, J2 Screw_Terminal_01x04, J3 Screw_Terminal_01x02, J4 Conn_ARM_JTAG_SWD_10, Q1 IRF6616, Q2 IRF6616, SW1 SW_Push, U1 4002B, U10 STM32F103CBUx, U7 LMR54406DBVR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

Commit message: Add files via upload
Parts:
- added J5: Screw_Terminal_01x02, TerminalBlock_MetzConnect:TerminalBlock_MetzConnect_Type055_RT01502HDWU_1x02_P5.00mm_Horizontal, F.Cu at (149.9, 71.1)
- moved U1 7.53 mm to (91.4, 73.7)
Changed lines of the file:
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@@
     (0 "F.Cu" signal)
     (31 "B.Cu" signal)
-    (32 "B.Adhes" user "B.Adhesive")
-    (33 "F.Adhes" user "F.Adhesive")
     (34 "B.Paste" user)
     (35 "F.Paste" user)
@@
     (38 "B.Mask" user)
     (39 "F.Mask" user)
-    (40 "Dwgs.User" user "User.Drawings")
-    (41 "Cmts.User" user "User.Comments")
-    (42 "Eco1.User" user "User.Eco1")
-    (43 "Eco2.User" user "User.Eco2")
     (44 "Edge.Cuts" user)
     (45 "Margin" user)
@@
     (48 "B.Fab" user)
     (49 "F.Fab" user)
-    (50 "User.1" user)
-    (51 "User.2" user)
-    (52 "User.3" user)
-    (53 "User.4" user)
-    (54 "User.5" user)
-    (55 "User.6" user)
-    (56 "User.7" user)
-    (57 "User.8" user)
     (58 "User.9" user)
   )
   (setup
+    (stackup
+      (layer "F.SilkS" (type "Top Silk Screen") (color "White"))
+      (layer "F.Paste" (type "Top Solder Paste"))
+      (layer "F.Mask" (type "Top Solder Mask") (color "Green") (thickness 0.01))
+      (layer "F.Cu" (type "copper") (thickness 0.035))
+      (layer "dielectric 1" (type "core") (thickness 1.51) (material "FR4") (epsilon_r 4.5) (loss_tangent 0.02))
+      (layer "B.Cu" (type "copper") (thickness 0.035))
+      (layer "B.Mask" (type "Bottom Solder Mask") (color "Green") (thickness 0.01))
+      (layer "B.Paste" (type "Bottom Solder Paste"))
+      (layer "B.SilkS" (type "Bottom Silk Screen") (color "White"))
+      (copper_finish "HAL lead-free")
+      (dielectric_constraints no)
+    )
     (pad_to_mask_clearance 0)
     (pcbplotparams
@@
   )
   (footprint "m12:m12con" (layer "F.Cu")
-    (at 97.565 78.045)
+    (at 91.44 73.66)
     (property "Sheetfile" "measurements_sch.kicad_sch")
     (property "Sheetname" "measurements")
     (attr through_hole)
-    (fp_text reference "U1" (at 0 -7.62 unlocked) (layer "F.SilkS")
-      (effects (font (size 1 1) (thickness 0.15)))
-    )
-    (fp_text value "4002B" (at 0 7.62 unlocked) (layer "F.Fab")
+    (fp_text reference "U1" (at 0 -12.7 unlocked) (layer "F.SilkS")
+      (effects (font (size 1 1) (thickness 0.15)))
+    )
+    (fp_text value "4002B" (at 0 12.7 unlocked) (layer "F.Fab")
       (effects (font (size 1 1) (thickness 0.15)))
     )
@@
         (xy -5.08 -10.16)
         (xy 5.08 -10.16)
-      ) (layer "F.SilkS") (width 0.12) (fill none))
+      ) (layer "F.SilkS") (width 0.2) (fill none))
     (pad "1" thru_hole circle (at -3.535 -3.535) (size 1.524 1.524) (drill 0.9) (layers *.Cu *.Mask)
       (net 60 "Net-(U1-Pad1)") (pinfunction "IN_M12") (pintype "power_out"))
@@
       (offset (xyz 0 0 0))
       (scale (xyz 1 1 1))
+      (rotate (xyz 0 0 0))
+    )
+  )
+  (footprint "TerminalBlock_MetzConnect:TerminalBlock_MetzConnect_Type055_RT01502HDWU_1x02_P5.00mm_Horizontal" (layer "F.Cu")
+    (at 149.86 71.12)
+    (descr "terminal block Metz Connect Type055_RT01502HDWU, 2 pins, pitch 5mm, size 10x8mm^2, drill diamater 1.3mm, pad diameter 2.5mm, see http://www.metz-connect.com/de/system/files/productfiles/Datenblatt_310551_RT015xxHDWU_OFF-022723S.pdf, script-generated using https://github.com/pointhi/kicad-footprint-generator/scripts/TerminalBlock_MetzConnect")
+    (tags "THT terminal block Metz Connect Type055_RT01502HDWU pitch 5mm size 10x8mm^2 drill 1.3mm pad 2.5mm")
+    (property "Sheetfile" "ultrasound_sch.kicad_sch")
+    (property "Sheetname" "communication")
+    (attr through_hole)
+    (fp_text reference "J5" (at 2.5 -5.06) (layer "F.SilkS")
+      (effects (font (size 1 1) (thickness 0.15)))
+    )
+    (fp_text value "Screw_Terminal_01x02" (at 2.5 5.06) (layer "F.Fab")
+      (effects (font (size 1 1) (thickness 0.15)))
+    )
+    (fp_text user "${REFERENCE}" (at 2.5 3) (layer "F.Fab")
+      (effects (font (size 1 1) (thickness 0.15)))
+    )
+    (fp_line (start -2.56 -4.06) (end -2.56 4.06) (layer "F.SilkS") (width 0.12))
+    (fp_line (start -2.8 4.3) (end -0.8 4.3) (layer "F.SilkS") (width 0.12))
+    (fp_line (start -2.56 2) (end 7.56 2) (layer "F.SilkS") (width 0.12))
+    (fp_line (start 7.56 -4.06) (end 7.56 4.06) (layer "F.SilkS") (width 0.12))
+    (fp_line (start -2.56 -4.06) (end 7.56 -4.06) (layer "F.SilkS") (width 0.12))
+    (fp_line (start 6.07 -1.275) (end 6.011 -1.216) (layer "F.SilkS") (width 0.12))
+    (fp_line (start -2.56 -2) (end 7.56 -2) (layer "F.SilkS") (width 0.12))
+    (fp_line (start 6.275 -1.069) (end 6.181 -0.976) (layer "F.SilkS") (width 0.12))
+    (fp_line (start 3.99 1.216) (end 3.931 1.274) (layer "F.SilkS") (width 0.12))
+    (fp_line (start -2.8 2.06) (end -2.8 4.3) (layer "F.SilkS") (width 0.12))
+    (fp_line (start 3.82 0.976) (end 3.726 1.069) (layer "F.SilkS") (width 0.12))
+    (fp_line (start -2.56 4.06) (end 7.56 4.06) (layer "F.SilkS") (width 0.12))
+    (fp_arc (start 0.029383 1.68045) (mid -0.392304 1.634281) (end -0.789 1.484) (layer "F.SilkS") (width 0.12))
+    (fp_arc (start -1.483953 0.789089) (mid -1.680708 0.00005) (end -1.484 -0.789) (layer "F.SilkS") (width 0.12))
+    (fp_arc (start -0.789089 -1.483953) (mid -0.00005 -1.680708) (end 0.789 -1.484) (layer "F.SilkS") (width 0.12))
+    (fp_arc (start 0.788712 1.483352) (mid 0.406429 1.630097) (end 0 1.68) (layer "F.SilkS") (width 0.12))
+    (fp_arc (start 1.483953 -0.789089) (mid 1.680708 -0.00005) (end 1.484 0.789) (layer "F.SilkS") (width 0.12))
+    (fp_circle (center 5 0) (end 6.68 0) (layer "F.SilkS") (width 0.12) (fill none))
+    (fp_line (start -3 -4.5) (end -3 4.5) (layer "F.CrtYd") (width 0.05))
+    (fp_line (start 8 -4.5) (end -3 -4.5) (layer "F.CrtYd") (width 0.05))
+    (fp_line (start -3 4.5) (end 8 4.5) (layer "F.CrtYd") (width 0.05))
+    (fp_line (start 8 4.5) (end 8 -4.5) (layer "F.CrtYd") (width 0.05))
+    (fp_line (start -2.5 -2) (end 7.5 -2) (layer "F.Fab") (width 0.1))
+    (fp_line (start 7.5 4) (end -0.5 4) (layer "F.Fab") (width 0.1))
+    (fp_line (start -2.5 2) (end -2.5 -4) (layer "F.Fab") (width 0.1))
+    (fp_line (start 7.5 -4) (end 7.5 4) (layer "F.Fab") (width 0.1))
+    (fp_line (start -2.5 2) (end 7.5 2) (layer "F.Fab") (width 0.1))
+    (fp_line (start -0.5 4) (end -2.5 2) (layer "F.Fab") (width 0.1))
+    (fp_line (start 6.138 -0.955) (end 4.046 1.138) (layer "F.Fab") (width 0.1))
+    (fp_line (start -2.5 -4) (end 7.5 -4) (layer "F.Fab") (width 0.1))
+    (fp_line (start 1.138 -0.955) (end -0.955 1.138) (layer "F.Fab") (width 0.1))
+    (fp_line (start 5.955 -1.138) (end 3.863 0.955) (layer "F.Fab") (width 0.1))
+    (fp_line (start 0.955 -1.138) (end -1.138 0.955) (layer "F.Fab") (width 0.1))
+    (fp_circle (center 5 0) (end 6.5 0) (layer "F.Fab") (width 0.1) (fill none))
+    (fp_circle (center 0 0) (end 1.5 0) (layer "F.Fab") (width 0.1) (fill none))
+    (pad "1" thru_hole rect (at 0 0) (size 2.5 2.5) (drill 1.3) (layers *.Cu *.Mask)
+      (net 58 "Net-(BZ1-Pad1)") (pinfunction "Pin_1") (pintype "passive"))
+    (pad "2" thru_hole circle (at 5 0) (size 2.5 2.5) (drill 1.3) (layers *.Cu *.Mask)
+      (net 1 "GND12V") (pinfunction "Pin_2") (pintype "passive"))
+    (model "${KICAD6_3DMODEL_DIR}/TerminalBlock_MetzConnect.3dshapes/TerminalBlock_MetzConnect_Type055_RT01502HDWU_1x02_P5.00mm_Horizontal.wrl"
+      (offset (xyz 0 0 0))
+      (scale (xyz 1 1 1))

Commit message: Add files via upload
Parts:
- moved R3 74.6 mm to (166.3, 109.0)
- moved R2 73.3 mm to (161.0, 109.0)
- moved C5 72.9 mm to (161.2, 107.0)
- moved R1 69.3 mm to (155.5, 109.0), turned to 180 degrees
- moved C3 57.8 mm to (149.5, 78.7)
- moved J4 56.0 mm to (162.0, 99.0)
- moved L3 47.6 mm to (114.5, 82.0)
- moved U1 45.7 mm to (131.0, 96.5)
- moved J5 45.0 mm to (162.6, 114.3)
- moved L2 37.8 mm to (115.5, 105.0)
- moved C1 37.3 mm to (149.5, 81.0)
- moved C4 36.8 mm to (144.8, 81.3)
- moved C2 36.8 mm to (144.8, 83.8)
- moved U10 36.5 mm to (155.0, 102.0)
- moved R7 36.4 mm to (163.6, 81.3)
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Routing:
- net GND12V: track 0.00 -> 89.8 mm, vias 0 -> 1
- net pres: track 0.00 -> 40.1 mm
- net 3.3V_GND: track 0.00 -> 38.5 mm, vias 0 -> 3
- net Net-(R12-Pad2): track 0.00 -> 32.4 mm
- net Net-(C5-Pad2): track 0.00 -> 29.7 mm
- net +3.3V: track 0.00 -> 29.1 mm, vias 0 -> 1
- net peri_power_2: track 0.00 -> 26.7 mm
- net RST: track 0.00 -> 26.2 mm, vias 0 -> 2
- net Net-(R10-Pad1): track 0.00 -> 15.0 mm
- net TDO: track 0.00 -> 13.8 mm, vias 0 -> 1
- net peri_power_1: track 0.00 -> 9.81 mm
- net Net-(BZ1-Pad1): track 0.00 -> 9.76 mm
- net acoustic: track 0.00 -> 7.29 mm
- net SWDIO: track 0.00 -> 6.85 mm
- net +5V: track 0.00 -> 5.73 mm
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
Commit message: Add files via upload
Parts:
- moved U7 37.1 mm to (116.4, 84.0)
- moved C12 36.0 mm to (120.0, 88.0)
- moved C10 28.5 mm to (150.2, 87.0)
- moved R10 28.0 mm to (144.0, 75.2), turned to 90 degrees
- moved C15 28.0 mm to (139.2, 103.0)
- moved R3 27.3 mm to (139.0, 108.5)
- moved R8 26.0 mm to (141.5, 95.5), turned to -90 degrees
- moved C14 23.9 mm to (136.5, 75.7), turned to 90 degrees
- moved R12 23.1 mm to (127.0, 93.5)
- moved R1 22.8 mm to (136.8, 96.0)
- moved R9 22.3 mm to (142.0, 80.5)
- moved R13 20.5 mm to (133.5, 98.5)
- moved C18 19.8 mm to (125.0, 87.5)
- moved L3 19.8 mm to (133.0, 89.0)
- moved D2 19.2 mm to (144.5, 108.1), turned to 90 degrees
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Routing:
- net GND12V: track 89.8 -> 0.00 mm, vias 1 -> 0
- net pres: track 40.1 -> 0.00 mm
- net 3.3V_GND: track 38.5 -> 0.00 mm, vias 3 -> 0
- net Net-(R12-Pad2): track 32.4 -> 0.00 mm
- net Net-(C5-Pad2): track 29.7 -> 0.00 mm
- net +3.3V: track 29.1 -> 0.00 mm, vias 1 -> 0
- net peri_power_2: track 26.7 -> 0.00 mm
- net RST: track 26.2 -> 0.00 mm, vias 2 -> 0
- net Net-(R10-Pad1): track 15.0 -> 0.00 mm
- net TDO: track 13.8 -> 0.00 mm, vias 1 -> 0
- net peri_power_1: track 9.81 -> 0.00 mm
- net Net-(BZ1-Pad1): track 9.76 -> 0.00 mm
- net acoustic: track 7.29 -> 0.00 mm
- net SWDIO: track 6.85 -> 0.00 mm
- net +5V: track 5.73 -> 0.00 mm
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