File: EECD-22-7.kicad_pcb (KiCad board)
At the start: 2 copper layers, 55 parts, among them J1 Screw_Terminal_01x03, J2 Screw_Terminal_01x04, J3 Screw_Terminal_01x02, J4 Conn_ARM_JTAG_SWD_10, J5 Screw_Terminal_01x02, Q1 IRF6616, Q2 IRF6616, SW1 SW_Push, U1 4002B, U10 STM32F103CBUx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

Commit message: Add files via upload
Parts:
- moved R1 57.1 mm to (144.8, 78.7)
- moved C3 57.1 mm to (148.8, 78.7)
- moved J4 56.0 mm to (162.0, 99.0)
- moved R3 52.7 mm to (144.5, 106.7)
- moved L3 48.0 mm to (114.3, 83.8)
- moved C5 46.0 mm to (130.3, 78.7)
- moved J5 45.0 mm to (162.6, 114.3)
- moved U1 44.4 mm to (129.5, 96.5)
- moved R2 44.0 mm to (130.3, 81.3)
- moved L2 39.6 mm to (114.3, 106.7)
- moved U10 38.3 mm to (156.8, 102.0)
- moved C1 36.8 mm to (148.8, 81.3)
- moved C4 36.8 mm to (144.8, 81.3)
- moved C2 36.8 mm to (144.8, 83.8)
- moved R7 36.4 mm to (163.6, 81.3)
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